File: hardware/pcb/SW-3240/SW-3240.kicad_pcb (KiCad board)
At the start: 2 copper layers, 0 parts

Commit message: many changes
Parts:
- added C1: 10uF, Capacitor_SMD:C_0603_1608Metric, F.Cu at (-76.2, 86.4)
- added C10: 470nF, Capacitor_SMD:C_0603_1608Metric, F.Cu at (-117.7, 132.4)
- added C11: 22nF, Capacitor_SMD:C_0603_1608Metric, F.Cu at (-133.5, 149.2)
- added C12: 1000uF, Capacitor_THT:C_Radial_D10.0mm_H20.0mm_P5.00mm, F.Cu at (-111.8, -35.6)
- added C13: 100nF, Capacitor_SMD:C_0603_1608Metric, F.Cu at (-133.5, 151.7)
- added C14: 1000uF, Capacitor_THT:C_Radial_D10.0mm_H20.0mm_P5.00mm, F.Cu at (-159.9, 54.6)
- added C15: 10uF, Capacitor_SMD:C_0603_1608Metric, F.Cu at (-137.5, 148.2)
- added C16: 1000uF, Capacitor_THT:C_Radial_D10.0mm_H20.0mm_P5.00mm, F.Cu at (-119.9, 134.9)
- added C17: 10uF, Capacitor_SMD:C_0603_1608Metric, F.Cu at (-137.5, 150.7)
- added C18: 10uF, Capacitor_SMD:C_0603_1608Metric, F.Cu at (-111.8, 127.8)
- added C19: 10uF, Capacitor_SMD:C_0603_1608Metric, F.Cu at (-115.9, 134.9)
- added C2: 100nF, Capacitor_SMD:C_0603_1608Metric, F.Cu at (-71.9, 63.5)
- added C20: 10uF, Capacitor_SMD:C_0603_1608Metric, F.Cu at (-119.9, 137.4)
- added C21: 100nF, Capacitor_SMD:C_0603_1608Metric, F.Cu at (50.8, 48.3)
- added C22: 100nF, Capacitor_SMD:C_0603_1608Metric, F.Cu at (24.6, 57.6)
- added C3: 100uF, Capacitor_SMD:C_0603_1608Metric, F.Cu at (-81.2, 96.0)
- added C4: 1uF, Capacitor_SMD:C_0603_1608Metric, F.Cu at (-5.16, 25.2)
- added C5: 10uF, Capacitor_SMD:C_0603_1608Metric, F.Cu at (-113.7, 131.9)
- added C6: 100nF, Capacitor_SMD:C_0603_1608Metric, F.Cu at (-107.8, 125.3)
- added C7: 10uF, Capacitor_SMD:C_0603_1608Metric, F.Cu at (-107.8, 127.8)
- added C8: 100uF, Capacitor_SMD:C_0603_1608Metric, F.Cu at (-106.7, -25.4)
- added C9: 100uF, Capacitor_SMD:C_0603_1608Metric, F.Cu at (-111.8, 125.3)
- added D1: 1N4004, Diode_SMD:D_SOD-123F, F.Cu at (-125.1, 129.1)
- added D2: SS34, Diode_SMD:D_SMC, F.Cu at (-71.1, -43.2)
- added D4: 1N4004, Diode_SMD:D_SOD-123F, F.Cu at (-141.2, 144.4)
- added D5: RED, LED_SMD:LED_0805_2012Metric, F.Cu at (-125.1, 125.8)
- added D6: RED, LED_SMD:LED_0805_2012Metric, F.Cu at (-132.2, 137.2)
- added D7: 1N4004, Diode_SMD:D_SOD-123F, F.Cu at (-129.9, 133.9)
- added H1: MountingHole, MountingHole:MountingHole_2.2mm_M2, F.Cu at (104.1, 198.1)
- added H2: MountingHole, MountingHole:MountingHole_2.2mm_M2, F.Cu at (-81.2, 85.8)
- added H3: MountingHole, MountingHole:MountingHole_2.2mm_M2, F.Cu at (-96.2, 102.9)
- added H4: MountingHole, MountingHole:MountingHole_2.2mm_M2, F.Cu at (-96.2, 108.8)
- added H5: MountingHole, MountingHole:MountingHole_2.2mm_M2, F.Cu at (276.9, 198.1)
- added H6: MountingHole, MountingHole:MountingHole_2.2mm_M2, F.Cu at (-81.2, 91.8)
- added J1: AUX_MIC_IN, Connector_PinHeader_2.54mm:PinHeader_1x02_P2.54mm_Vertical, F.Cu at (154.9, 174.0)
- added J10: RESET/FLASH, Connector_PinHeader_2.54mm:PinHeader_2x02_P2.54mm_Vertical, F.Cu at (136.4, 189.4)
- added J11: PWR, SaawLib:BarrelJack_CUI_PJ-102AH_Horizontal, F.Cu at (-131.1, 61.2)
- added J12: BAT, Connector_JST:JST_XH_B2B-XH-A_1x02_P2.50mm_Vertical, F.Cu at (116.8, 223.5)
- added J13: CH_1, SaawLib:STX-3100-5N, F.Cu at (223.5, 196.5)
- added J14: CH_2, SaawLib:STX-3100-5N, F.Cu at (243.8, 196.5)
- added J15: CH_3, SaawLib:STX-3100-5N, F.Cu at (264.2, 196.5)
- added J16: CH_4, SaawLib:STX-3100-5N, F.Cu at (70.7, 47.8)
- added J2: AUX_LINE_IN, Connector_PinHeader_2.54mm:PinHeader_1x04_P2.54mm_Vertical, F.Cu at (175.3, 196.5)
- added J3: MIC, SaawLib:STX-3100-5N, F.Cu at (160.3, 196.5)
- added J4: LINE IN, SaawLib:STX-3100-5N, F.Cu at (-29.0, 73.0)
- added J5: ESPFlash, Connector_PinHeader_2.54mm:PinHeader_2x03_P2.54mm_Vertical, F.Cu at (-19.1, 68.6)
- added J6: JTAG, Connector_PinHeader_2.54mm:PinHeader_2x05_P2.54mm_Vertical, F.Cu at (-58.4, 49.5)
- added J7: I2C, Connector_PinHeader_2.54mm:PinHeader_1x04_P2.54mm_Vertical, F.Cu at (105.5, 141.7)
- added J8: MIC_IN_R, Connector_PinHeader_2.54mm:PinHeader_1x01_P2.54mm_Vertical, F.Cu at (185.4, 191.4)
- added J9: FP_IO, Connector_JST:JST_XH_B6B-XH-A_1x06_P2.50mm_Vertical, F.Cu at (154.9, 182.9)
- added JP1: SolderJumper_3_Bridged123, SaawLib:SolderJumper-3_P1.3mm_Bridged123_Pad1.0x1.5mm_NumberLabels, F.Cu at (-86.0, 96.9)
- added JP2: TRI_PHASE, Connector_PinHeader_2.54mm:PinHeader_2x01_P2.54mm_Vertical, F.Cu at (193.0, 191.4)
- added JP3: TRI_PHASE, Connector_PinHeader_2.54mm:PinHeader_2x01_P2.54mm_Vertical, F.Cu at (213.4, 191.4)
- added JP4: TRI_PHASE, Connector_PinHeader_2.54mm:PinHeader_2x01_P2.54mm_Vertical, F.Cu at (233.7, 191.4)
- added JP5: TRI_PHASE, Connector_PinHeader_2.54mm:PinHeader_2x01_P2.54mm_Vertical, F.Cu at (254.0, 191.4)
- added L1: 100uH, Inductor_THT:L_Toroid_Vertical_L24.6mm_W15.5mm_P11.44mm_Pulse_KM-4, F.Cu at (-67.9, -22.9)
- added R1: 2.7K, Resistor_SMD:R_0603_1608Metric, F.Cu at (-72.2, 88.9)
- added R10: 10K, Resistor_SMD:R_0603_1608Metric, F.Cu at (-124.9, 143.6)
- added R11: 1K, Resistor_SMD:R_0603_1608Metric, F.Cu at (-132.9, 144.1)
- added R12: 100K, Resistor_SMD:R_0603_1608Metric, F.Cu at (-129.5, 149.2)
- added R13: 9K, Resistor_SMD:R_0603_1608Metric, F.Cu at (-137.5, 153.2)
- added R14: 1K, Resistor_SMD:R_0603_1608Metric, F.Cu at (-116.3, 129.4)
- added R15: 470, Resistor_SMD:R_0603_1608Metric, F.Cu at (-123.9, 136.1)
- added R16: 10K, Resistor_SMD:R_0603_1608Metric, F.Cu at (-121.7, 132.4)
- added R17: 2.7K, Resistor_SMD:R_0603_1608Metric, F.Cu at (-128.9, 144.0)
- added R2: 2.7K, Resistor_SMD:R_0603_1608Metric, F.Cu at (-51.0, 67.8)
- added R3: 10K, Resistor_SMD:R_0603_1608Metric, F.Cu at (-76.2, 91.4)
- added R4: 10k, Resistor_SMD:R_0603_1608Metric, F.Cu at (-55.0, 70.3)
- added R5: 10k, Resistor_SMD:R_0603_1608Metric, F.Cu at (-98.4, 113.4)
- added R6: 2.7K, Resistor_SMD:R_0603_1608Metric, F.Cu at (-76.2, 88.9)
- added R7: 2.7K, Resistor_SMD:R_0603_1608Metric, F.Cu at (-55.0, 67.8)
- added R8: 100K, Resistor_SMD:R_0603_1608Metric, F.Cu at (-124.3, 141.1)
- added R9: 84.5K, Resistor_SMD:R_0603_1608Metric, F.Cu at (-128.9, 146.5)
- added SW1: PWR_SW, Button_Switch_THT:SW_E-Switch_EG2219_DPDT_Angled, F.Cu at (-38.1, 58.4)
- added TP1: EN, TestPoint:TestPoint_THTPad_D2.0mm_Drill1.0mm, F.Cu at (-137.0, 144.9)
- added TP2: 5V, TestPoint:TestPoint_THTPad_D2.0mm_Drill1.0mm, F.Cu at (-127.9, 137.4)
- added TP3: 14V, TestPoint:TestPoint_THTPad_D2.0mm_Drill1.0mm, F.Cu at (-120.3, 129.2)
- added TP4: 9V, TestPoint:TestPoint_THTPad_D2.0mm_Drill1.0mm, F.Cu at (-141.5, 147.9)
- added TP5: 13.5V, TestPoint:TestPoint_THTPad_D2.0mm_Drill1.0mm, F.Cu at (-125.7, 132.8)
- added TP6: 12V, TestPoint:TestPoint_THTPad_D2.0mm_Drill1.0mm, F.Cu at (-115.9, 126.1)
- added TP7: 3.3V, TestPoint:TestPoint_THTPad_D2.0mm_Drill1.0mm, F.Cu at (-141.5, 152.0)
- added TP8: 3.3V_ALT, TestPoint:TestPoint_THTPad_D2.0mm_Drill1.0mm, F.Cu at (-132.4, 140.8)
- added U1: SW-32MA, SaawLib:SW-32MA_Socket, F.Cu at (165.2, 163.5)
- added U10: LMR14050, Package_SO:TI_SO-PowerPAD-8, F.Cu at (-138.9, 139.7)
- added U11: NCP1117-3.3, Package_TO_SOT_SMD:SOT-223-3_TabPin2, F.Cu at (-48.9, 40.6)
- added U12: NCP1117-3.3, Package_TO_SOT_SMD:SOT-223-3_TabPin2, F.Cu at (-132.1, 116.8)
- added U2: MCP4728, Package_SO:MSOP-10_3x3mm_P0.5mm, F.Cu at (215.9, 172.7)
- added U3: ESP32-WROOM-32D, RF_Module:ESP32-WROOM-32, F.Cu at (215.9, 157.5)
- added U4: Channel 1, SaawLib:SW-32MO_Socket, F.Cu at (188.0, 153.3)
- added U5: Channel 2, SaawLib:SW-32MO_Socket, F.Cu at (213.4, 153.3)
- added U6: Channel 3, SaawLib:SW-32MO_Socket, F.Cu at (238.8, 153.3)
- added U7: Channel 4, SaawLib:SW-32MO_Socket, F.Cu at (264.2, 153.3)
- added U8: LM2576-5, Package_TO_SOT_SMD:TO-263-5_TabPin3, F.Cu at (-89.7, -45.7)
- added U9: LM2941, Package_TO_SOT_SMD:TO-263-5_TabPin3, F.Cu at (-121.0, 40.9)
Other:
- board outline added: 177.8 x 157.5 mm
