File: hardware/pcb/SW-3240/SW-3240.kicad_pcb (KiCad board)
At the start: 2 copper layers, 177.8 x 157.5 mm, 94 parts, among them J1 AUX_MIC_IN, J10 RESET/FLASH, J11 PWR, J12 BAT, J13 CH_1, J14 CH_2, J15 CH_3, J16 CH_4, J2 AUX_LINE_IN, J3 MIC, J4 LINE IN, J5 ESPFlash, J6 JTAG, J7 I2C, J8 MIC_IN_R, J9 FP_IO, SW1 PWR_SW, U1 SW-32MA, U10 LMR14050, U11 NCP1117-3.3, U12 NCP1117-3.3, U2 MCP4728, U3 ESP32-WROOM-32D, U4 Channel 1, U5 Channel 2, U6 Channel 3, U7 Channel 4, U8 LM2576-5, U9 LM2941

Commit message: major changes
Parts:
- removed JP5: TRI_PHASE, Connector_PinHeader_2.54mm:PinHeader_2x01_P2.54mm_Vertical
- removed TP1: EN, TestPoint:TestPoint_THTPad_D2.0mm_Drill1.0mm
- removed TP8: 3.3V_ALT, TestPoint:TestPoint_THTPad_D2.0mm_Drill1.0mm
- removed U10: LMR14050, Package_SO:TI_SO-PowerPAD-8
- removed U11, U12: NCP1117-3.3, Package_TO_SOT_SMD:SOT-223-3_TabPin2
- removed U7: Channel 4, SaawLib:SW-32MO_Socket
- removed U8: LM2576-5, Package_TO_SOT_SMD:TO-263-5_TabPin3
- removed U9: LM2941, Package_TO_SOT_SMD:TO-263-5_TabPin3
- added C23: 100nF, Capacitor_SMD:C_0603_1608Metric, F.Cu at (102.9, 88.4)
- added D3: SSB44-E3, Diode_SMD:D_SMB, F.Cu at (232.4, 54.5)
- added F1: 1A, Fuse:Fuse_BelFuse_0ZRE0005FF_L8.3mm_W3.8mm, F.Cu at (79.2, 109.5)
- added F2: 4A, Fuse:Fuse_BelFuse_0ZRE0016FF_L9.9mm_W3.8mm, F.Cu at (77.6, 100.9)
- added H10: MountingHole, MountingHole:MountingHole_2.2mm_M2, F.Cu at (241.3, 90.2)
- added H11: MountingHole, MountingHole:MountingHole_2.2mm_M2, F.Cu at (154.9, 90.2)
- added H12: MountingHole, MountingHole:MountingHole_2.2mm_M2, F.Cu at (68.6, 90.2)
- added H7: MountingHole, MountingHole:MountingHole_2.2mm_M2, F.Cu at (154.9, 147.3)
- added H8: MountingHole, MountingHole:MountingHole_2.2mm_M2, F.Cu at (101.6, 33.0)
- added H9: MountingHole, MountingHole:MountingHole_2.2mm_M2, F.Cu at (208.3, 33.0)
- added J17: CH_2, SaawLib:STX-3100-5N, F.Cu at (190.5, 146.1)
- added J18: CH_3, SaawLib:STX-3100-5N, F.Cu at (210.8, 146.1)
- added J19: CH_4, SaawLib:STX-3100-5N, F.Cu at (231.1, 146.1)
- added L2: 15uH, Inductor_SMD:L_Bourns_SRR1260, F.Cu at (90.8, 39.6)
- added Q1: BSS138, Package_TO_SOT_SMD:SOT-23, F.Cu at (148.1, 96.3)
- added Q2: BSS138, Package_TO_SOT_SMD:SOT-23, F.Cu at (148.0, 100.8)
- added R18: 10K, Resistor_SMD:R_0603_1608Metric, F.Cu at (197.4, 102.8)
- added R19: 4.7K, Resistor_SMD:R_0603_1608Metric, F.Cu at (197.4, 108.5)
- added R20: 1K, Resistor_SMD:R_0603_1608Metric, F.Cu at (210.4, 55.2)
- added R21: 1K, Resistor_SMD:R_0603_1608Metric, F.Cu at (210.4, 58.1)
- added Y1: 16MHz, Crystal:Crystal_HC49-4H_Vertical, F.Cu at (166.6, 108.7)
- C1, C5: value 10uF -> 100nF
- C10: value 470nF -> 10uF; footprint Capacitor_SMD:C_0603_1608Metric -> Capacitor_SMD:C_1210_3225Metric
- C11: value 22nF -> 10uF; footprint Capacitor_SMD:C_0603_1608Metric -> Capacitor_SMD:C_1210_3225Metric
- C12: value 1000uF -> 10uF; footprint Capacitor_THT:C_Radial_D10.0mm_H20.0mm_P5.00mm -> Capacitor_SMD:C_1210_3225Metric
- C13: value 100nF -> 10uF; footprint Capacitor_SMD:C_0603_1608Metric -> Capacitor_SMD:C_1210_3225Metric
- C14: value 1000uF -> 470nF; footprint Capacitor_THT:C_Radial_D10.0mm_H20.0mm_P5.00mm -> Capacitor_SMD:C_0603_1608Metric
- C15: value 10uF -> 10nF
- C16: value 1000uF -> 10nF; footprint Capacitor_THT:C_Radial_D10.0mm_H20.0mm_P5.00mm -> Capacitor_SMD:C_0603_1608Metric
- C17: value 10uF -> 100uF; footprint Capacitor_SMD:C_0603_1608Metric -> Capacitor_THT:C_Radial_D8.0mm_H11.5mm_P3.50mm
- C18: value 10uF -> 180uF; footprint Capacitor_SMD:C_0603_1608Metric -> Capacitor_SMD:CP_Elec_10x7.9
- C19: value 10uF -> 330uF; footprint Capacitor_SMD:C_0603_1608Metric -> Capacitor_SMD:CP_Elec_10x12.6
- C2, C21, C22: value 100nF -> 10uF
- C20: value 10uF -> 330uF; footprint Capacitor_SMD:C_0603_1608Metric -> Capacitor_THT:C_Radial_D8.0mm_H11.5mm_P3.50mm
- C3: value 100uF -> 100nF
- C4: value 1uF -> 10uF
- C6: value 100nF -> 22pF
- C7: value 10uF -> 22pF
- C8, C9: footprint Capacitor_SMD:C_0603_1608Metric -> Capacitor_THT:C_Radial_D8.0mm_H11.5mm_P3.50mm
- D1: value 1N4004 -> LED; footprint Diode_SMD:D_SOD-123F -> LED_SMD:LED_0603_1608Metric
- D2: value SS34 -> SSB44-E3; footprint Diode_SMD:D_SMC -> Diode_SMD:D_SMB
- D4: value 1N4004 -> SSB44-E3; footprint Diode_SMD:D_SOD-123F -> Diode_SMD:D_SMB
- D5: value RED -> SSB44-E3; footprint LED_SMD:LED_0805_2012Metric -> Diode_SMD:D_SMB
- D6: value RED -> GREEN; footprint LED_SMD:LED_0805_2012Metric -> LED_SMD:LED_0603_1608Metric
- D7: value 1N4004 -> BLUE; footprint Diode_SMD:D_SOD-123F -> LED_SMD:LED_0603_1608Metric
- J10: value RESET/FLASH -> PWR; footprint Connector_PinHeader_2.54mm:PinHeader_2x02_P2.54mm_Vertical -> SaawLib:BarrelJack_CUI_PJ-102AH_Horizontal
- J11: value PWR -> BAT; footprint SaawLib:BarrelJack_CUI_PJ-102AH_Horizontal -> Connector_JST:JST_XH_B2B-XH-A_1x02_P2.50mm_Vertical
- J12: value BAT -> Channel 1; footprint Connector_JST:JST_XH_B2B-XH-A_1x02_P2.50mm_Vertical -> SaawLib:SW-32MO_Socket
- J13: value CH_1 -> Channel 2; footprint SaawLib:STX-3100-5N -> SaawLib:SW-32MO_Socket
- J14: value CH_2 -> Channel 3; footprint SaawLib:STX-3100-5N -> SaawLib:SW-32MO_Socket
- J15: value CH_3 -> Channel 4; footprint SaawLib:STX-3100-5N -> SaawLib:SW-32MO_Socket
- J16: value CH_4 -> CH_1
- J5: value ESPFlash -> ICSP
- J6: value JTAG -> FP_IO; footprint Connector_PinHeader_2.54mm:PinHeader_2x05_P2.54mm_Vertical -> Connector_JST:JST_XH_B8B-XH-A_1x08_P2.50mm_Vertical
- J7: value I2C -> MIC_IN_R; footprint Connector_PinHeader_2.54mm:PinHeader_1x04_P2.54mm_Vertical -> Connector_PinHeader_2.54mm:PinHeader_1x01_P2.54mm_Vertical
- J8: value MIC_IN_R -> FTDI; footprint Connector_PinHeader_2.54mm:PinHeader_1x01_P2.54mm_Vertical -> Connector_PinHeader_2.54mm:PinHeader_1x06_P2.54mm_Vertical
- J9: value FP_IO -> SW-32MA; footprint Connector_JST:JST_XH_B6B-XH-A_1x06_P2.50mm_Vertical -> SaawLib:SW-32MA_Socket
- JP1: value SolderJumper_3_Bridged123 -> JP1; footprint SaawLib:SolderJumper-3_P1.3mm_Bridged123_Pad1.0x1.5mm_NumberLabels -> Connector_PinHeader_2.54mm:PinHeader_2x01_P2.54mm_Vertical
- JP2: value TRI_PHASE -> JP2
- JP3: value TRI_PHASE -> JP3
- JP4: value TRI_PHASE -> JP4
- L1: value 100uH -> 15uH; footprint Inductor_THT:L_Toroid_Vertical_L24.6mm_W15.5mm_P11.44mm_Pulse_KM-4 -> Inductor_SMD:L_Bourns_SRR1260
- R1, R17: value 2.7K -> 1K
- R10: value 10K -> 100K
- R11: value 1K -> 10K
- R12: value 100K -> 1K
- R13: value 9K -> 10K
- R14: value 1K -> 1.5K
- R15: value 470 -> 10K
- R16: value 10K -> 3.24K
- R2, R6, R7: value 2.7K -> 4.7K
- R3: value 10K -> 4.7K
- R4: value 10k -> 10K
- R5: value 10k -> 4.7K
- R8: value 100K -> 4.7K
- R9: value 84.5K -> 10K
- TP2: value 5V -> 14V; footprint TestPoint:TestPoint_THTPad_D2.0mm_Drill1.0mm -> TestPoint:TestPoint_Pad_D1.5mm
- TP3: value 14V -> 9.2V; footprint TestPoint:TestPoint_THTPad_D2.0mm_Drill1.0mm -> TestPoint:TestPoint_Pad_D1.5mm
- TP4: value 9V -> 5V; footprint TestPoint:TestPoint_THTPad_D2.0mm_Drill1.0mm -> TestPoint:TestPoint_Pad_D1.5mm
- TP5: value 13.5V -> VBAT; footprint TestPoint:TestPoint_THTPad_D2.0mm_Drill1.0mm -> TestPoint:TestPoint_Pad_D1.5mm
- TP6, TP7: footprint TestPoint:TestPoint_THTPad_D2.0mm_Drill1.0mm -> TestPoint:TestPoint_Pad_D1.5mm
- U1: value SW-32MA -> MCP4728; footprint SaawLib:SW-32MA_Socket -> Package_SO:MSOP-10_3x3mm_P0.5mm
- U2: value MCP4728 -> ATmega328PB-AU; footprint Package_SO:MSOP-10_3x3mm_P0.5mm -> Package_QFP:TQFP-32_7x7mm_P0.8mm
- U3: value ESP32-WROOM-32D -> TPS5430DDA; footprint RF_Module:ESP32-WROOM-32 -> Package_SO:TI_SO-PowerPAD-8_ThermalVias
- U4: value Channel 1 -> TPS5430DDA; footprint SaawLib:SW-32MO_Socket -> Package_SO:TI_SO-PowerPAD-8_ThermalVias
- U5: value Channel 2 -> LM2941; footprint SaawLib:SW-32MO_Socket -> Package_TO_SOT_SMD:TO-263-5_TabPin3
- U6: value Channel 3 -> NCP1117-3.3; footprint SaawLib:SW-32MO_Socket -> Package_TO_SOT_SMD:SOT-223-3_TabPin2
- moved C15 384.2 mm to (233.7, 49.1)
- moved R13 374.8 mm to (221.6, 45.8), turned to 90 degrees
- moved R10 358.0 mm to (221.6, 53.7), turned to 90 degrees
- moved C8 355.9 mm to (236.9, 67.7), turned to 90 degrees
- moved TP3 353.6 mm to (220.3, 34.5), turned to -90 degrees
- moved C12 351.2 mm to (225.2, 63.4)
- moved C10 350.7 mm to (225.2, 58.7)
- moved D7 348.0 mm to (210.3, 61.0), turned to 180 degrees
- moved R14 347.1 mm to (221.6, 50.0), turned to 90 degrees
- moved C18 336.2 mm to (214.0, 45.0), turned to -90 degrees
- moved H2 326.8 mm to (241.3, 33.0)
- moved R9 325.7 mm to (194.6, 108.5), turned to 90 degrees
- moved L1 304.9 mm to (230.5, 39.6), turned to 180 degrees
- moved H6 298.2 mm to (215.9, 66.0)
- moved R5 290.5 mm to (192.0, 108.5), turned to 90 degrees
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Connections:
- C1 pad 1: +3V3 -> /RESET
- C1 pad 2: GND -> Net-(C1-Pad2)
- C10 pad 1: Net-(C10-Pad1) -> GND
- C10 pad 2: GND -> +12V
- C11 pad 2: Net-(C11-Pad2) -> +12V
- C12 pad 1: +5V -> GND
- C12 pad 2: GND -> +12V
- C13 pad 1: Net-(C13-Pad1) -> GND
- C13 pad 2: Net-(C13-Pad2) -> +12V
- C15 pad 1: +5V -> Net-(C15-Pad1)
- C15 pad 2: GND -> Net-(C15-Pad2)
- C16 pad 2: GND -> Net-(C16-Pad2)
- C17 pad 1: +5V -> Net-(C17-Pad1)
- C18 pad 1: +5V -> +9V
- C19 pad 1: +3V3 -> +5V
- C2 pad 1: +3V3 -> +5V
- C20 pad 1: /+3.3V_FP -> Net-(C20-Pad1)
- C21 pad 1: +3V3 -> +5V
- C22 pad 1: /+3.3V_FP -> +3V3
- C3 pad 1: +3V3 -> +5V
- C4 pad 1: /EN -> +5V
- C5 pad 1: +3V3 -> +5V
- C6 pad 1: +3V3 -> Net-(C6-Pad1)
- C7 pad 1: +12V -> Net-(C7-Pad1)
- D1 pad 1: Net-(C10-Pad1) -> GND
- D1 pad 2: /PSU/VIN -> Net-(D1-Pad2)
- D2 pad 1: Net-(D2-Pad1) -> Net-(C14-Pad1)
- D2 pad 2: GND -> /PSU/VIN
- D4 pad 1: Net-(D4-Pad1) -> Net-(C16-Pad2)
- D4 pad 2: Net-(C14-Pad1) -> GND
- D5 pad 1: GND -> Net-(D5-Pad1)
- D5 pad 2: Net-(D5-Pad2) -> Net-(C17-Pad1)
- D7 pad 1: Net-(C16-Pad1) -> GND
- D7 pad 2: GND -> Net-(D7-Pad2)
- J10 pad 1: GND -> /PSU/VIN
- J10 pad 2: /EN -> GND
- J10 pad 3: GND -> (no net)
- J11 pad 1: /PSU/VIN -> /PSU/VBAT
- J12 pad 1: /PSU/VBAT -> +9V
- J12 pad 2: GND -> +5V
- J16 pad S: Net-(J16-PadS) -> Net-(J12-Pad8)
- J16 pad T: Net-(J16-PadT) -> Net-(J12-Pad10)
- J5 pad 1: /EN -> /MISO
- J5 pad 2: +3V3 -> +5V
- J5 pad 3: /TXD -> /SCK
- J5 pad 4: GND -> /MOSI
- J5 pad 5: /RXD -> /RESET
- J5 pad 6: /IO0 -> GND
- J6 pad 1: +3V3 -> GND
- J6 pad 2: /MTMS -> +5V
- J6 pad 3: GND -> +3V3
- J6 pad 4: /MTCK -> /SCL_3V3
- J6 pad 5: unconnected-(J6-Pad5) -> /SDA_3V3
- J6 pad 6: /MTDO -> /LINE_RIGHT
- J6 pad 7: unconnected-(J6-Pad7) -> /LINE_LEFT
- J6 pad 8: /MTDI -> /MIC
- J7 pad 1: GND -> Net-(J3-PadR)
- J8 pad 1: Net-(J3-PadR) -> Net-(C1-Pad2)
- J9 pad 1: GND -> +3V3
- J9 pad 2: /+3.3V_FP -> GND
- J9 pad 3: /SCL -> /MIC
- J9 pad 4: /SDA -> /LINE_LEFT
- J9 pad 5: /CH_PSU_EN -> /LINE_RIGHT
- J9 pad 6: /VBAT_SENSE -> Net-(J3-PadT)
- JP1 pad 1: Net-(JP1-Pad1) -> Net-(J12-Pad9)
- JP1 pad 2: +3V3 -> Net-(J16-PadR)
- JP2 pad 1: Net-(JP2-Pad1) -> Net-(J13-Pad9)
- JP2 pad 2: Net-(J13-PadR) -> Net-(J17-PadR)
- JP3 pad 1: Net-(JP3-Pad1) -> Net-(J14-Pad9)
- JP3 pad 2: Net-(J14-PadR) -> Net-(J18-PadR)
- JP4 pad 1: Net-(JP4-Pad1) -> Net-(J15-Pad9)
- JP4 pad 2: Net-(J15-PadR) -> Net-(J19-PadR)
- L1 pad 1: Net-(D2-Pad1) -> Net-(C15-Pad2)
- L1 pad 2: +5V -> +9V
- R1 pad 1: +3V3 -> /SCK
- R1 pad 2: /DAC_SCL -> Net-(D1-Pad2)
- R10 pad 1: Net-(C14-Pad1) -> /CH_PSU_EN
- R10 pad 2: Net-(R10-Pad2) -> GND
- R11 pad 1: Net-(R10-Pad2) -> Net-(C17-Pad1)
- R11 pad 2: GND -> Net-(R11-Pad2)
- R12 pad 1: +9V -> Net-(R11-Pad2)
- R12 pad 2: Net-(R12-Pad2) -> GND
- R13 pad 1: Net-(R12-Pad2) -> Net-(R13-Pad1)
- R13 pad 2: GND -> +9V
- R14 pad 1: Net-(D5-Pad2) -> GND
- R14 pad 2: +9V -> Net-(R13-Pad1)
- R15 pad 1: Net-(D6-Pad2) -> Net-(R15-Pad1)
- R15 pad 2: +3V3 -> +5V
- R16 pad 1: +12V -> GND
- R16 pad 2: /VBAT_SENSE -> Net-(R15-Pad1)
- R17 pad 1: /VBAT_SENSE -> Net-(D6-Pad2)
- R17 pad 2: GND -> +5V
- R2 pad 2: /DAC_SDA -> /SDA_3V3
- R3 pad 1: GND -> +3V3
- R3 pad 2: Net-(R3-Pad2) -> /SCL_3V3
- R4 pad 1: /IO0 -> +5V
- R4 pad 2: +3V3 -> /RESET
- R5 pad 1: /EN -> +5V
- R5 pad 2: +3V3 -> /DAC_SCL
- R6 pad 1: Net-(JP1-Pad3) -> +5V
- R6 pad 2: /SCL -> /SDA
- R7 pad 1: Net-(JP1-Pad1) -> +5V
- R7 pad 2: /SDA -> /DAC_SDA
- R8 pad 1: /CH_PSU_EN -> +5V
- R8 pad 2: GND -> /SCL
- R9 pad 1: Net-(R9-Pad1) -> GND
- R9 pad 2: GND -> Net-(R9-Pad2)
- SW1 pad 1: Net-(C16-Pad1) -> +12V
- SW1 pad 2: +12V -> Net-(C20-Pad1)
- SW1 pad 3: (no net) -> unconnected-(SW1-Pad3)
- SW1 pad 4: (no net) -> unconnected-(SW1-Pad4)
- SW1 pad 5: (no net) -> unconnected-(SW1-Pad5)
- SW1 pad 6: (no net) -> unconnected-(SW1-Pad6)
- TP2 pad 1: +5V -> Net-(C17-Pad1)
- TP3 pad 1: Net-(C14-Pad1) -> +9V
- TP4 pad 1: +9V -> +5V
- TP5 pad 1: Net-(C16-Pad1) -> Net-(C20-Pad1)
- U1 pad 1: +3V3 -> +5V
- U1 pad 10: Net-(J2-Pad2) -> GND
- U1 pad 2: GND -> /DAC_SCL
- U1 pad 3: /MIC -> /DAC_SDA
- U1 pad 4: /LINE_LEFT -> Net-(R9-Pad2)
- U1 pad 5: /LINE_RIGHT -> unconnected-(U1-Pad5)
- U1 pad 6: Net-(J3-PadT) -> /CHA_LEVEL
- U1 pad 7: Net-(J1-Pad1) -> /CHB_LEVEL
- U1 pad 8: Net-(J4-PadT) -> /CHC_LEVEL
- U1 pad 9: Net-(J4-PadR) -> /CHD_LEVEL
- U2 pad 1: +3V3 -> /CHA_PULSE_A
- U2 pad 10: GND -> /CHB_I_SENSE
- U2 pad 2: /DAC_SCL -> /CHA_PULSE_B
- U2 pad 4: Net-(R3-Pad2) -> +5V
- U2 pad 5: unconnected-(U2-Pad5) -> GND
- U2 pad 6: /CHA_I_LIMIT -> /DAC_SCL
- U2 pad 7: /CHB_I_LIMIT -> Net-(C7-Pad1)
- U2 pad 8: /CHC_I_LIMIT -> Net-(C6-Pad1)
- U2 pad 9: /CHD_I_LIMIT -> /CHB_PULSE_A
- U3 pad 1: GND -> Net-(C15-Pad1)
- U3 pad 2: +3V3 -> unconnected-(U3-Pad2)
- U3 pad 3: /EN -> unconnected-(U3-Pad3)
- U3 pad 4: /CHD_I_SENSE -> Net-(R13-Pad1)
- U3 pad 5: /CHC_I_SENSE -> /CH_PSU_EN
- U3 pad 6: /CHB_I_SENSE -> GND
- U3 pad 7: /CHA_I_SENSE -> +12V
- U3 pad 8: /DAC_SDA -> Net-(C15-Pad2)
- U3 pad 9: /CHC_PULSE_B -> GND
- U4 pad 1: +9V -> Net-(C16-Pad1)
- U4 pad 2: +3V3 -> unconnected-(U4-Pad2)
- U4 pad 3: GND -> unconnected-(U4-Pad3)
- U4 pad 4: /CHA_I_SENSE -> Net-(R15-Pad1)
- U4 pad 5: /CHA_I_LIMIT -> unconnected-(U4-Pad5)
- U4 pad 6: /CHA_PULSE_A -> GND
- U4 pad 7: /CHA_PULSE_B -> +12V
- U4 pad 8: Net-(J13-PadS) -> Net-(C16-Pad2)
- U4 pad 9: Net-(JP2-Pad1) -> GND
- U5 pad 1: +9V -> Net-(R11-Pad2)
- U5 pad 2: +3V3 -> GND
- U5 pad 4: /CHB_I_SENSE -> Net-(C14-Pad1)
- U5 pad 5: /CHB_I_LIMIT -> Net-(C17-Pad1)
- U6 pad 1: +9V -> GND
- U6 pad 3: GND -> +5V
Routing:
- net +5V: track 0.00 -> 318.7 mm, vias 0 -> 6
- net +9V: track 0.00 -> 128.9 mm, vias 0 -> 3
- net /SCK: track 0.00 -> 108.1 mm, vias 0 -> 4
- net /MOSI: track 0.00 -> 93.9 mm, vias 0 -> 3
- net /CH_PSU_EN: track 0.00 -> 93.2 mm, vias 0 -> 2
- net /MISO: track 0.00 -> 93.2 mm, vias 0 -> 3
- net /CHA_LEVEL: track 0.00 -> 88.9 mm, vias 0 -> 2
- net /RESET: track 0.00 -> 85.6 mm, vias 0 -> 2
- net +3V3: track 0.00 -> 82.4 mm, vias 0 -> 2
- net /CHA_I_SENSE: track 0.00 -> 74.5 mm
- net /TXD: track 0.00 -> 67.6 mm, vias 0 -> 1
- net /RXD: track 0.00 -> 66.1 mm, vias 0 -> 1
- net /CHB_I_SENSE: track 0.00 -> 57.7 mm, vias 0 -> 1
- net /CHD_PULSE_A: track 0.00 -> 57.6 mm
- net /CHD_PULSE_B: track 0.00 -> 57.0 mm
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- added copper zone on B.Cu, net +12V
- added copper zone on F.Cu, net +12V
- added copper zone on F.Cu, net +5V
- added copper zone on F.Cu, net +9V
- added copper zone on B.Cu, net GND
- added copper zone on F.Cu, net GND
- added copper zone on F.Cu, net Net-(C15-Pad2)
- added copper zone on F.Cu, net Net-(C16-Pad2)
- added copper zone on B.Cu, net Net-(C20-Pad1)
- added copper zone on F.Cu, net Net-(C20-Pad1)
Other:
- board size 177.8 x 157.5 mm -> 177.8 x 119.4 mm
- board text added: "JLCJLCJLCJLC"
