File: hardware/pcb/modules/audio/SW-32MA1/SW-32MA1.kicad_pcb (KiCad board)
At the start: 2 copper layers, 44.6 x 15.2 mm, 24 parts, among them U1 Opamp_Quad, U2 SW-32MA

Commit message: major changes
Routing:
- net /MIC: track 12.9 -> 12.3 mm
