File: hardware/pcb/modules/control/SW-32MC1/SW-32MC1.kicad_pcb (KiCad board)
At the start: 2 copper layers, 0 parts

Commit message: major changes
Parts:
- added BZ1: Buzzer, Buzzer_Beeper:Buzzer_12x9.5RM7.6, B.Cu at (94.0, 94.6)
- added C1: 10nF, Capacitor_SMD:C_0603_1608Metric, B.Cu at (159.2, 98.4)
- added C10: 100nF, Capacitor_SMD:C_0603_1608Metric, B.Cu at (231.0, 116.2)
- added C11: 100nF, Capacitor_SMD:C_0603_1608Metric, B.Cu at (251.3, 116.2)
- added C2: 10nF, Capacitor_SMD:C_0603_1608Metric, B.Cu at (155.7, 98.4)
- added C3: 10uF, Capacitor_SMD:C_0603_1608Metric, B.Cu at (151.6, 84.5)
- added C4: 100nF, Capacitor_SMD:C_0603_1608Metric, B.Cu at (151.6, 87.6)
- added C5: 10nF, Capacitor_SMD:C_0603_1608Metric, B.Cu at (158.1, 85.1)
- added C6: 100nF, Capacitor_SMD:C_0603_1608Metric, B.Cu at (142.1, 116.2)
- added C7: 100nF, Capacitor_SMD:C_0603_1608Metric, B.Cu at (157.3, 116.2)
- added C8: 100nF, Capacitor_SMD:C_0603_1608Metric, B.Cu at (190.4, 116.2)
- added C9: 100nF, Capacitor_SMD:C_0603_1608Metric, B.Cu at (210.7, 116.2)
- added D1: LED, LED_SMD:LED_0603_1608Metric, B.Cu at (125.1, 109.9)
- added D10: WS2812D, SaawLib:WS2812D-F5, F.Cu at (251.5, 118.1)
- added D2: D_Small, Diode_SMD:D_SOD-123F, B.Cu at (96.0, 102.9)
- added D3: D, Diode_SMD:D_SOD-123F, B.Cu at (126.4, 114.3)
- added D4: WS2812D, SaawLib:WS2812D-F5, B.Cu at (119.4, 113.0)
- added D5: WS2812D, SaawLib:WS2812D-F5, F.Cu at (142.2, 118.1)
- added D6: WS2812D, SaawLib:WS2812D-F5, F.Cu at (157.5, 118.1)
- added D7: WS2812D, SaawLib:WS2812D-F5, F.Cu at (190.5, 118.1)
- added D8: WS2812D, SaawLib:WS2812D-F5, F.Cu at (210.8, 118.1)
- added D9: WS2812D, SaawLib:WS2812D-F5, F.Cu at (231.1, 118.1)
- added H1: MountingHole, MountingHole:MountingHole_2.2mm_M2, F.Cu at (175.3, 95.2)
- added H2: MountingHole, MountingHole:MountingHole_2.2mm_M2, F.Cu at (259.1, 109.2)
- added H3: MountingHole, MountingHole:MountingHole_2.2mm_M2, F.Cu at (94.0, 109.2)
- added H4: MountingHole, MountingHole:MountingHole_2.2mm_M2, F.Cu at (94.0, 83.8)
- added H5: MountingHole, MountingHole:MountingHole_2.2mm_M2, F.Cu at (259.1, 83.8)
- added J1: JTAG, Connector_IDC:IDC-Header_2x05_P2.54mm_Vertical, B.Cu at (152.4, 108.5)
- added J2: ESPFlash, Connector_IDC:IDC-Header_2x03_P2.54mm_Vertical, B.Cu at (107.9, 103.4)
- added J3: OLED, SaawLib:OLED_I2C_1.3, F.Cu at (119.4, 84.5)
- added J4: FP_IO, Connector_JST:JST_XH_B8B-XH-A_1x08_P2.50mm_Vertical, B.Cu at (165.1, 85.7)
- added J5: I2C, Connector_PinHeader_2.54mm:PinHeader_1x04_P2.54mm_Vertical, B.Cu at (99.7, 84.5)
- added JP1: SolderJumper_3_Bridged12, Jumper:SolderJumper-3_P1.3mm_Bridged12_Pad1.0x1.5mm_NumberLabels, B.Cu at (114.9, 90.1)
- added JP2: SolderJumper_3_Bridged12, Jumper:SolderJumper-3_P1.3mm_Bridged12_Pad1.0x1.5mm_NumberLabels, B.Cu at (111.1, 90.1)
- added JP4: SolderJumper_3_Bridged123, SaawLib:SolderJumper-3_P1.3mm_Bridged123_Pad1.0x1.5mm_NumberLabels, B.Cu at (106.0, 90.8)
- added Q1: Q_NMOS_DGS, Package_TO_SOT_SMD:SOT-23, B.Cu at (108.7, 96.8)
- added R1: 10K, Resistor_SMD:R_0603_1608Metric, B.Cu at (159.2, 95.2)
- added R10: 10K, Resistor_SMD:R_0603_1608Metric, B.Cu at (113.1, 97.8)
- added R11: 2.7K, Resistor_SMD:R_0603_1608Metric, B.Cu at (107.3, 87.9)
- added R12: 10K, Resistor_SMD:R_0603_1608Metric, B.Cu at (150.5, 101.6)
- added R2: 10K, Resistor_SMD:R_0603_1608Metric, B.Cu at (155.8, 95.2)
- added R3: 10k, Resistor_SMD:R_0603_1608Metric, B.Cu at (121.9, 100.3)
- added R4: 10K, Resistor_SMD:R_0603_1608Metric, B.Cu at (154.9, 84.3)
- added R5: 10k, Resistor_SMD:R_0603_1608Metric, B.Cu at (129.0, 109.9)
- added R8: 2.7K, Resistor_SMD:R_0603_1608Metric, B.Cu at (104.8, 87.9)
- added R9: 10, Resistor_SMD:R_0603_1608Metric, B.Cu at (113.1, 94.9)
- added RV1: 20K, Potentiometer_THT:Potentiometer_Bourns_PTV09A-1_Single_Vertical, F.Cu at (193.1, 102.6)
- added RV2: 20K, Potentiometer_THT:Potentiometer_Bourns_PTV09A-1_Single_Vertical, F.Cu at (213.4, 102.6)
- added RV3: 20K, Potentiometer_THT:Potentiometer_Bourns_PTV09A-1_Single_Vertical, F.Cu at (233.7, 102.6)
- added RV4: 20K, Potentiometer_THT:Potentiometer_Bourns_PTV09A-1_Single_Vertical, F.Cu at (254.0, 102.6)
- added SW1: PEC11R-4225F-S0024, SaawLib:Rotary_Encoder_Switched_PEC11R, F.Cu at (151.8, 95.0)
- added SW2: DNP, Button_Switch_SMD:SW_Push_1P1T_NO_6x6mm_H9.5mm, F.Cu at (172.7, 104.1)
- added U1: ESP32-WROOM-32D, RF_Module:ESP32-WROOM-32, B.Cu at (135.5, 97.2)
Routing:
- net +3V3: track 0.00 -> 280.2 mm, vias 0 -> 5
- net +5V: track 0.00 -> 212.0 mm
- net /LVL_D: track 0.00 -> 118.4 mm
- net /LVL_C: track 0.00 -> 97.6 mm
- net /LVL_B: track 0.00 -> 76.7 mm
- net /ENC_B: track 0.00 -> 63.4 mm
- net /LVL_A: track 0.00 -> 56.6 mm
- net /ENC_A: track 0.00 -> 55.9 mm
- net /MAIN_SCL: track 0.00 -> 49.8 mm, vias 0 -> 2
- net /LINE_LEFT: track 0.00 -> 46.9 mm, vias 0 -> 3
- net /MIC: track 0.00 -> 46.4 mm, vias 0 -> 3
- net /MAIN_SDA: track 0.00 -> 44.5 mm, vias 0 -> 3
- net /EN: track 0.00 -> 41.0 mm, vias 0 -> 1
- net /LINE_RIGHT: track 0.00 -> 39.1 mm, vias 0 -> 3
- net /ENC_SW: track 0.00 -> 37.9 mm, vias 0 -> 1
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- added copper zone on B.Cu, net GND
- added copper zone on F.Cu, net GND
Other:
- board outline added: 170.2 x 40.7 mm
- board text added: "JLCJLCJLCJLC"
