File: hardware/pcb/modules/output/SW-32MO10/SW-32MO10.kicad_pcb (KiCad board)
At the start: 2 copper layers, 65 x 23.8 mm, 35 parts, among them Q1 NTF2955, Q2 DMN2041L, Q3 DMN2041L, T1 42TL004-RC, U1 SW-32MO, U2 TLV272IS-13

Commit message: major changes
Parts:
- removed C5: 1uF, Capacitor_SMD:C_0603_1608Metric
- removed R1: 10k, Resistor_SMD:R_0603_1608Metric
- moved C9 3.46 mm to (112.3, 81.0), turned to 180 degrees
- moved R2 2.63 mm to (103.6, 81.9)
- moved R3 2.63 mm to (103.6, 80.0)
- moved C7 1.65 mm to (112.2, 79.0)
- moved R5 0.63 mm to (108.1, 80.0)
Connections:
- U2 pad 3: Net-(C5-Pad1) -> /I_LIMIT
Routing:
- net Net-(C5-Pad1): track 6.32 -> 0.00 mm
- net /I_LIMIT: track 7.31 -> 11.6 mm
- net Net-(R2-Pad1): track 5.82 -> 7.92 mm
- net +9V: track 9.40 -> 7.38 mm
- net Net-(R3-Pad1): track 5.41 -> 6.21 mm
- net Net-(Q1-Pad1): track 12.7 -> 12.1 mm
