File: hardware/pcb/modules/output/SW-32MO10/SW-32MO10.kicad_sch (KiCad schematic)
At the start: 35 parts, among them Q1 NTF2955, Q2 DMN2041L, Q3 DMN2041L, T1 42TL004-RC, U1 SW-32MO, U2 TLV272IS-13

Commit message: update pdf
Other:
- moved on the sheet: C5, C7, C9, R1, R2, R3, U2A

Commit message: major changes
Parts:
- removed C5: 1uF, Capacitor_SMD:C_0603_1608Metric, symbol Device:C
- removed R1: 10k, Resistor_SMD:R_0603_1608Metric, symbol Device:R
Connections:
- net I_LIMIT: now also U2.3 (+)
Other:
- note added: "AV = 1.47"
- note added: "Board-to-Board Connector"
Changed lines of the file:
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@@
     (comment 4 "A single channel e-stim module driver board for the SW-3240")
-  )
-  (junction (at 64.77 91.44) (diameter 0) (color 0 0 0 0)
   )
   (junction (at 86.36 68.58) (diameter 0) (color 0 0 0 0)
@@
     (stroke (width 0) (type default) (color 0 0 0 0))
   )
-  (wire (pts (xy 30.48 91.44) (xy 53.34 91.44))
-    (stroke (width 0) (type default) (color 0 0 0 0))
-  )
   (wire (pts (xy 124.46 54.61) (xy 124.46 78.74))
     (stroke (width 0) (type default) (color 0 0 0 0))
@@
     (stroke (width 0) (type default) (color 0 0 0 0))
   )
-  (wire (pts (xy 64.77 91.44) (xy 64.77 95.25))
-    (stroke (width 0) (type default) (color 0 0 0 0))
-  )
   (wire (pts (xy 21.59 29.21) (xy 21.59 31.75))
     (stroke (width 0) (type default) (color 0 0 0 0))
@@
     (stroke (width 0) (type default) (color 0 0 0 0))
   )
-  (wire (pts (xy 60.96 91.44) (xy 64.77 91.44))
+  (wire (pts (xy 48.26 91.44) (xy 101.6 91.44))
     (stroke (width 0) (type default) (color 0 0 0 0))
   )
@@
     (stroke (width 0) (type default) (color 0 0 0 0))
   )
-  (wire (pts (xy 64.77 91.44) (xy 101.6 91.44))
-    (stroke (width 0) (type default) (color 0 0 0 0))
-  )
   (wire (pts (xy 151.13 31.75) (xy 151.13 34.29))
     (stroke (width 0) (type default) (color 0 0 0 0))
@@
   )
   (wire (pts (xy 137.16 44.45) (xy 124.46 44.45))
-    (stroke (width 0) (type default) (color 0 0 0 0))
-  )
-  (wire (pts (xy 64.77 102.87) (xy 64.77 106.68))
     (stroke (width 0) (type default) (color 0 0 0 0))
   )
@@
     (effects (font (size 1.27 1.27)) (justify left bottom))
   )
+  (text "AV = 1.47\n" (at 119.38 93.98 0)
+    (effects (font (size 1.27 1.27)) (justify left bottom))
+  )
   (text "Shunt Amplifier" (at 182.88 124.46 0)
     (effects (font (size 2 2)) (justify left bottom))
@@
     (effects (font (size 2 2)) (justify left bottom))
   )
+  (text "Board-to-Board Connector" (at 40.64 172.72 0)
+    (effects (font (size 1 1)) (justify left bottom))
+  )
   (label "OUTA" (at 74.93 158.75 180)
     (effects (font (size 1.27 1.27)) (justify right bottom))
@@
     (effects (font (size 1.27 1.27)) (justify right bottom))
   )
-  (label "I_LIMIT" (at 30.48 91.44 0)
+  (label "I_LIMIT" (at 48.26 91.44 0)
     (effects (font (size 1.27 1.27)) (justify left bottom))
   )
@@
     (pin "2")
     (pin "3")
-  )
-  (symbol (lib_id "Device:R") (at 57.15 91.44 270) (unit 1)
-    (in_bom yes) (on_board yes)
-    (property "Reference" "R1" (id 0) (at 57.15 86.36 90))
-    (property "Value" "10k" (id 1) (at 57.15 88.9 90))
-    (property "Footprint" "Resistor_SMD:R_0603_1608Metric" (id 2) (at 57.15 89.662 90)
-      (effects (font (size 1.27 1.27)) hide)
-    )
-    (property "Datasheet" "~" (id 3) (at 57.15 91.44 0)
-      (effects (font (size 1.27 1.27)) hide)
-    )
-    (property "MPN" "RC0603FR-0710KL" (id 4) (at 57.15 91.44 0)
-      (effects (font (size 1.27 1.27)) hide)
-    )
-    (pin "1")
-    (pin "2")
   )
   (symbol (lib_id "SaawLib:Transformer_SP_SS") (at 254 31.75 0) (unit 1)
@@
     (pin "2")
   )
-  (symbol (lib_id "power:GND") (at 64.77 106.68 0) (unit 1)
-    (in_bom yes) (on_board yes)
-    (property "Reference" "#PWR05" (id 0) (at 64.77 113.03 0)
-      (effects (font (size 1.27 1.27)) hide)
-    )
-    (property "Value" "GND" (id 1) (at 64.77 110.49 0))
-    (property "Footprint" "" (id 2) (at 64.77 106.68 0)
-      (effects (font (size 1.27 1.27)) hide)
-    )
-    (property "Datasheet" "" (id 3) (at 64.77 106.68 0)
-      (effects (font (size 1.27 1.27)) hide)
-    )
-    (pin "1")
-  )
   (symbol (lib_id "Device:R") (at 116.84 78.74 270) (unit 1)
     (in_bom yes) (on_board yes)
@@
     (pin "1")
   )
-  (symbol (lib_id "Device:C") (at 64.77 99.06 0) (unit 1)
-    (in_bom yes) (on_board yes)
-    (property "Reference" "C5" (id 0) (at 67.31 97.79 0)
-      (effects (font (size 1.27 1.27)) (justify left))
-    )
-    (property "Value" "1uF" (id 1) (at 67.31 100.33 0)
-      (effects (font (size 1.27 1.27)) (justify left))
-    )
-    (property "Footprint" "Capacitor_SMD:C_0603_1608Metric" (id 2) (at 65.7352 102.87 0)
-      (effects (font (size 1.27 1.27)) hide)
-    )
-    (property "Datasheet" "~" (id 3) (at 64.77 99.06 0)
-      (effects (font (size 1.27 1.27)) hide)
-    )
-    (property "MPN" "CL10B105KA8NFNC" (id 4) (at 64.77 99.06 0)
-      (effects (font (size 1.27 1.27)) hide)
-    )
-    (pin "1")
-    (pin "2")
-  )
   (symbol (lib_id "Amplifier_Operational:LMC6482") (at 238.76 139.7 0) (mirror x) (unit 2)
     (in_bom yes) (on_board yes)
@@
       (reference "#PWR04") (unit 1) (value "GND") (footprint "")
     )
-    (path "/7a847c3e-054e-4b54-8c0d-630102587bf6"
-      (reference "#PWR05") (unit 1) (value "GND") (footprint "")
-    )
     (path "/70fc40a7-475b-433d-a18b-69aa1344dad6"
       (reference "#PWR06") (unit 1) (value "+9V") (footprint "")
@@
       (reference "C4") (unit 1) (value "22uF") (footprint "Capacitor_SMD:C_1210_3225Metric")
     )
-    (path "/c9f94645-4d60-4ad4-b313-45216a860369"
-      (reference "C5") (unit 1) (value "1uF") (footprint "Capacitor_SMD:C_0603_1608Metric")
-    )
     (path "/a9ac2053-4d34-4641-a149-08a0ee7619e4"
       (reference "C6") (unit 1) (value "22uF") (footprint "Capacitor_SMD:C_1210_3225Metric")
@@
       (reference "Q3") (unit 1) (value "DMN2041L") (footprint "Package_TO_SOT_SMD:SOT-23")
     )
-    (path "/14ac3eae-3659-4ed0-a21a-c916eee4dc86"
-      (reference "R1") (unit 1) (value "10k") (footprint "Resistor_SMD:R_0603_1608Metric")
-    )
     (path "/0b9f2f8b-1340-44b1-bba2-d6506992d5aa"
