File: hardware/pcb/front_panel/SW-3240FP.kicad_sch (KiCad schematic)
At the start: 53 parts, among them J1 JTAG, J2 ESPFlash, J3 OLED, J4 FP_IO, J5 I2C, Q1 DMN2040U, SW1 PEC11R-4225F-S0024, SW2 DNP, U1 ESP32-WROOM-32D

Commit message: refactor
Other:
- title: SW-32MC1 -> SW-3240: Front Panel
Changed lines of the file:
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@@
   (paper "A4")
   (title_block
-    (title "SW-32MC1")
+    (title "SW-3240: Front Panel")
     (date "2022-02-02")
     (rev "1")

Commit message: redesign
Parts:
- removed C3: 10uF, Capacitor_SMD:C_0603_1608Metric, symbol Device:C_Small
- removed C6: 100nF, Capacitor_SMD:C_0603_1608Metric, symbol Device:C_Small
- removed D1: LED, LED_SMD:LED_0603_1608Metric, symbol Device:LED
- removed D2: D_Small, Diode_SMD:D_SOD-123F, symbol Device:D_Small
- removed D4: WS2812D, SaawLib:WS2812D-F5, symbol SaawLib:WS2812D
- removed H1: MountingHole, MountingHole:MountingHole_2.2mm_M2, symbol Mechanical:MountingHole
- removed J1: JTAG, Connector_IDC:IDC-Header_2x05_P2.54mm_Vertical, symbol Connector_Generic:Conn_02x05_Odd_Even
- removed J2: ESPFlash, Connector_IDC:IDC-Header_2x03_P2.54mm_Vertical, symbol Connector_Generic:Conn_02x03_Odd_Even
- removed J3: OLED, SaawLib:OLED_I2C_1.3, symbol SaawLib:OLED_MODULE_I2C
- removed J4: FP_IO, Connector_JST:JST_XH_B8B-XH-A_1x08_P2.50mm_Vertical, symbol Connector_Generic:Conn_01x08
- removed J5: I2C, Connector_PinHeader_2.54mm:PinHeader_1x04_P2.54mm_Vertical, symbol Connector_Generic:Conn_01x04
- removed JP1, JP2: SolderJumper_3_Bridged12, Jumper:SolderJumper-3_P1.3mm_Bridged12_Pad1.0x1.5mm_NumberLabels, symbol Jumper:SolderJumper_3_Bridged12
- removed JP3: SolderJumper_3_Bridged123, SaawLib:SolderJumper-3_P1.3mm_Bridged123_Pad1.0x1.5mm_NumberLabels, symbol Jumper:SolderJumper_3_Bridged123
- removed Q1: DMN2040U, Package_TO_SOT_SMD:SOT-23, symbol Device:Q_NMOS_SGD
- removed R10, R9: 10K, Resistor_SMD:R_0603_1608Metric, symbol Device:R
- removed R3, R5: 10k, Resistor_SMD:R_0603_1608Metric, symbol Device:R
- removed R6, R7: 2.7K, Resistor_SMD:R_0603_1608Metric, symbol Device:R
- removed R8: 10, Resistor_SMD:R_0603_1608Metric, symbol Device:R
- removed SW2: DNP, Button_Switch_SMD:SW_Push_1P1T_NO_6x6mm_H9.5mm, symbol Switch:SW_Push
- removed U1: ESP32-WROOM-32D, RF_Module:ESP32-WROOM-32, symbol RF_Module:ESP32-WROOM-32D
- added J1: MAIN_BOARD, Connector_PinHeader_2.54mm:PinHeader_2x08_P2.54mm_Vertical, symbol Connector_Generic:Conn_02x08_Odd_Even
- BZ1: MOUSER (none) -> 497-IE122303-1; MPN (none) -> IE122303-1
- C1, C2: LCSC (none) -> C1589; MOUSER (none) -> 187-CL10B103KB8NNNC; MPN (none) -> CL10B103KB8NNNC
- C3: renamed from C5; LCSC (none) -> C1589; MOUSER (none) -> 187-CL10B103KB8NNNC; MPN (none) -> CL10B103KB8NNNC
- C4: LCSC (none) -> C1591; MOUSER (none) -> 187-CL10B104KB8NNNC; MPN (none) -> CL10B104KB8NNNC
- C5: renamed from C7; LCSC (none) -> C1591; MOUSER (none) -> 187-CL10B104KB8NNNC; MPN (none) -> CL10B104KB8NNNC
- C6: renamed from C8; LCSC (none) -> C1591; MOUSER (none) -> 187-CL10B104KB8NNNC; MPN (none) -> CL10B104KB8NNNC
- C7: renamed from C9; LCSC (none) -> C1591; MOUSER (none) -> 187-CL10B104KB8NNNC; MPN (none) -> CL10B104KB8NNNC
- C8: renamed from C10; LCSC (none) -> C1591; MOUSER (none) -> 187-CL10B104KB8NNNC; MPN (none) -> CL10B104KB8NNNC
- C9: renamed from C11; LCSC (none) -> C1591; MOUSER (none) -> 187-CL10B104KB8NNNC; MPN (none) -> CL10B104KB8NNNC
- D1: renamed from D3; value D -> MBR120; symbol Device:D -> Device:D_Schottky; LCSC (none) -> C236132; MOUSER (none) -> 863-MBR120ESFT1G; MPN (none) -> MBR120ESFT1G
- R1, R2: LCSC (none) -> C98220; MOUSER (none) -> 603-RC0603FR-0710KL; MPN (none) -> RC0603FR-0710KL
- R3: renamed from R4; LCSC (none) -> C98220; MOUSER (none) -> 603-RC0603FR-0710KL; MPN (none) -> RC0603FR-0710KL
- RV1, RV2, RV3, RV4: MPN (none) -> PTV09A-40xxS-A203
- SW1: MPN PEC11R-4215F-S0024 -> PEC11R-42xxK-S0024
- renumbered D5 to D2, D6 to D3, D7 to D4, D8 to D5, D9 to D6, D10 to D7, H2 to H1, H3 to H2, H4 to H3, H5 to H4
Connections:
- net +3V3: now also J1.3 (Pin_3); no longer BZ1.1 (-), C4.1
- net +5V: now also J1.5 (Pin_5); no longer D2.2 (VCC)
- net BUZZER: now also BZ1.1 (-), J1.15 (Pin_15)
- net ENC_A: now also J1.7 (Pin_7)
- net ENC_B: now also J1.9 (Pin_9)
- net ENC_SW: now also J1.11 (Pin_11)
- net GND: now also BZ1.2 (+), C4.1, J1.1 (Pin_1); no longer C4.2
- net LED_DATA: now also D2.4 (DIN), J1.13 (Pin_13)
- net at D1.1 (K): now also C4.2, D2.2 (VCC)
- net LVL_A renamed LVL_1
- net LVL_1: now also J1.2 (Pin_2)
- net LVL_B renamed LVL_2
- net LVL_2: now also J1.4 (Pin_4)
- net LVL_C renamed LVL_3
- net LVL_3: now also J1.6 (Pin_6)
- net LVL_D renamed LVL_4
- net LVL_4: now also J1.8 (Pin_8)
- no-connect marks 11 -> 5
Other:
- note added: "First LED acts as level shifter V_{IH} = 0.7V_{DD}"
- note added: "max 40mA GPIO (buzzer 20mA @ 3.3V)"
- note added: "~0.6V"
- note removed: "1.5" OLED Module"
- note removed: "Back/Multi Button"
- note removed: "Boot Strapping Pins: IO 0,2,5,12,15 LED: IO2 I2C: IO 21, 22 JTAG: IO12-15"
- note removed: "Connectors"
- note removed: "ESP32"
- note removed: "First LED acts as level shifter & is hidden"
- note removed: "I2C"
- note removed: "I2C Pull-Ups"
- note removed: "JTAG IO12-15"
- note removed: "~0.7V"
- moved on the sheet: BZ1, C1, C2, C3, C5, C6, C7, C8, C9, D1, D2, D3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
