File: hardware/pcb/front_panel/SW-324FP.kicad_sch (KiCad schematic)
At the start: 30 parts, among them J1 MAIN_BOARD, SW1 PEC11R-4225F-S0024

Commit message: fix comments
Parts:
- added C1, C6: 100nF, Capacitor_SMD:C_0603_1608Metric, symbol Device:C_Small
- added C5: 10uF, Capacitor_SMD:C_0603_1608Metric, symbol Device:C_Small
- added D1: D_Small, symbol Device:D_Small
- added Q1: Q_NMOS_GSD, symbol Device:Q_NMOS_GSD
- added R2, R3: 10K, Resistor_SMD:R_0603_1608Metric, symbol Device:R_Small
- added R6: 330, Resistor_SMD:R_0603_1608Metric, symbol Device:R
- added R7: 10K, Resistor_SMD:R_0603_1608Metric, symbol Device:R
- added SW2: BTN1, symbol Switch:SW_Push
- added SW3: BTN2, symbol Switch:SW_Push
- added SW4: BTN3, symbol Switch:SW_Push
- added SW5: BTN4, symbol Switch:SW_Push
- added U1: PCF8574, Package_SO:TSSOP-20_4.4x6.5mm_P0.65mm, symbol Interface_Expansion:PCF8574
- added U2: PCF8591, symbol Interface_Expansion:PCF8591
- J1: footprint Connector_PinHeader_2.54mm:PinHeader_2x08_P2.54mm_Vertical -> Connector_IDC:IDC-Header_2x04_P2.54mm_Vertical; symbol Connector_Generic:Conn_02x08_Odd_Even -> Connector_Generic:Conn_02x04_Odd_Even
- renumbered C7 to C10, C8 to C11, C9 to C12, C1 to C2, C2 to C3, C3 to C4, C4 to C7, C5 to C8, C6 to C9, D1 to D2, D2 to D3, D3 to D4, D4 to D5, D5 to D6, D6 to D7, D7 to D8, R2 to R4, R3 to R5
Connections:
- net +3V3: now also BZ1.1 (-), C1.1, C5.1, C6.1, D1.1 (K), R2.1, R3.1, U1.16 (VDD), U2.14 (VREF), U2.16 (VDD)
- net BUZZER: now also R6.1, U1.4 (P0); no longer BZ1.1 (-), J1.15 (Pin_15)
- net ENC_A: now also U1.11 (P6); no longer J1.7 (Pin_7)
- net ENC_B: now also U1.12 (P7); no longer J1.9 (Pin_9)
- net ENC_SW: now also U1.10 (P5); no longer J1.11 (Pin_11)
- net GND: now also C1.2, C5.2, C6.2, Q1.2 (S), R7.1, SW2.1, SW3.1, SW4.1, SW5.1, U1.1 (A0), U1.8 (VSS), U2.12 (EXT), U2.13 (AGND), U2.5 (A0), U2.6 (A1), U2.7 (A2), U2.8 (VSS); no longer BZ1.2 (+)
- net LED_DATA: now also J1.6 (Pin_6); no longer J1.13 (Pin_13)
- net LVL_1: no longer names the net of RV1.2
- net LVL_1: now also U2.2 (AIN1); no longer J1.2 (Pin_2)
- net LVL_2: no longer names the net of RV2.2
- net LVL_2: now also U2.3 (AIN2); no longer J1.4 (Pin_4)
- net LVL_3: no longer names the net of RV3.2
- net LVL_3: now also U2.1 (AIN0); no longer J1.6 (Pin_6)
- net LVL_4: no longer names the net of RV4.2
- net LVL_4: now also U2.4 (AIN3); no longer J1.8 (Pin_8)
- new net: R2.2, U1.2 (A1)
- new net: R3.2, U1.3 (A2)
- new net: BZ1.2 (+), D1.2 (A), Q1.3 (D)
- new net: Q1.1 (G), R6.2, R7.2
- new net BTN1: SW2.2, U1.5 (P1)
- new net BTN2: SW3.2, U1.6 (P2)
- new net BTN3: SW4.2, U1.7 (P3)
- new net BTN4: SW5.2, U1.9 (P4)
- new net INT1: J1.7 (Pin_7), U1.13 (~{INT})
- new net INT2: J1.8 (Pin_8)
- new net SCL: J1.4 (Pin_4), U1.14 (SCL), U2.10 (SCL)
- new net SDA: J1.2 (Pin_2), U1.15 (SDA), U2.9 (SDA)
- no-connect marks 5 -> 3
Other:
- note added: "Port Expander"
- note removed: "max 40mA GPIO (buzzer 20mA @ 3.3V)"
- title: SW-3240: Front Panel -> SW-324: Front Panel
- moved on the sheet: BZ1, C10, C11, C12, C2, C3, C4, C7, C8, C9, D2, D3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
