File: hardware/pcb/main_board/SW-3240.kicad_sch (KiCad schematic)
At the start: 57 parts, among them J1 AUX_MIC_IN, J10 PWR, J11 BAT, J12 Channel 1, J13 Channel 2, J14 Channel 3, J15 Channel 4, J16 CH_1, J17 CH_2, J18 CH_3, J19 CH_4, J2 AUX_LINE_IN, J3 MIC, J4 LINE IN, J5 ICSP, J6 FP_IO, J7 MIC_IN_R, J8 FTDI, J9 SW-32MA, Q1 BSS138, Q2 BSS138, U1 MCP4728, U2 ATmega328PB-AU, Y1 16MHz

Commit message: refactor
Other:
- title: SW-3240 -> SW-3240: Main Board
Changed lines of the file:
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@@
   (paper "A4")
   (title_block
-    (title "SW-3240")
+    (title "SW-3240: Main Board")
     (date "2022-04-07")
     (rev "1")
     (company "saawsm")
-    (comment 1 "See connector FP_IO and front panel board (e.g. SW-32MC1).")
+    (comment 1 "See connector FP_IO and front panel board.")
     (comment 2 "Requires an I2C connection for control.")
     (comment 3 "The main board for the SW-3240.")

Commit message: update part numbers
Parts:
- C6, C7: LCSC (none) -> C1653; MOUSER (none) -> 187-CL10C220JB8NNNC; MPN (none) -> CL10C220JB8NNNC
- J1, J12, J13, J14, J15, J2, J5, J8, J9, JP1, JP2, JP3, JP4: now left out of the parts list
- Q1, Q2: LCSC (none) -> C890265; MOUSER (none) -> 512-BSS138L; MPN BSS138 -> BSS138L
- Y1: MOUSER (none) -> 815-ABL-16-B2; MPN (none) -> ABL-16.000MHZ-B2

Commit message: redesign
Parts:
- removed C3, C5: 100nF, Capacitor_SMD:C_0603_1608Metric, symbol Device:C_Small
- removed C4: 10uF, Capacitor_SMD:C_0603_1608Metric, symbol Device:C_Small
- removed C6, C7: 22pF, Capacitor_SMD:C_0603_1608Metric, symbol Device:C_Small
- removed D1: LED, LED_SMD:LED_0603_1608Metric, symbol Device:LED
- removed J1: AUX_MIC_IN, Connector_PinHeader_2.54mm:PinHeader_1x02_P2.54mm_Vertical, symbol Connector_Generic:Conn_01x02
- removed J10: PWR, SaawLib:BarrelJack_CUI_PJ-102AH_Horizontal, symbol Connector:Barrel_Jack
- removed J11: BAT, Connector_JST:JST_XH_B2B-XH-A_1x02_P2.50mm_Vertical, symbol Connector:Screw_Terminal_01x02
- removed J12: Channel 1, SaawLib:SW-32MO_Socket, symbol SaawLib:SW-32MO
- removed J13: Channel 2, SaawLib:SW-32MO_Socket, symbol SaawLib:SW-32MO
- removed J14: Channel 3, SaawLib:SW-32MO_Socket, symbol SaawLib:SW-32MO
- removed J15: Channel 4, SaawLib:SW-32MO_Socket, symbol SaawLib:SW-32MO
- removed J16: CH_1, SaawLib:STX-3100-5N, symbol Connector:AudioJack3_SwitchTR
- removed J17: CH_2, SaawLib:STX-3100-5N, symbol Connector:AudioJack3_SwitchTR
- removed J18: CH_3, SaawLib:STX-3100-5N, symbol Connector:AudioJack3_SwitchTR
- removed J19: CH_4, SaawLib:STX-3100-5N, symbol Connector:AudioJack3_SwitchTR
- removed J2: AUX_LINE_IN, Connector_PinHeader_2.54mm:PinHeader_1x04_P2.54mm_Vertical, symbol Connector_Generic:Conn_01x04
- removed J5: ICSP, Connector_PinHeader_2.54mm:PinHeader_2x03_P2.54mm_Vertical, symbol Connector_Generic:Conn_02x03_Odd_Even
- removed J6: FP_IO, Connector_JST:JST_XH_B8B-XH-A_1x08_P2.50mm_Vertical, symbol Connector_Generic:Conn_01x08
- removed J7: MIC_IN_R, Connector_PinHeader_2.54mm:PinHeader_1x01_P2.54mm_Vertical, symbol Connector_Generic:Conn_01x01
- removed J8: FTDI, Connector_PinHeader_2.54mm:PinHeader_1x06_P2.54mm_Vertical, symbol Connector_Generic:Conn_01x06
- removed JP1: JP1, Connector_PinHeader_2.54mm:PinHeader_2x01_P2.54mm_Vertical, symbol Jumper:Jumper_2_Open
- removed JP2: JP2, Connector_PinHeader_2.54mm:PinHeader_2x01_P2.54mm_Vertical, symbol Jumper:Jumper_2_Open
- removed JP3: JP3, Connector_PinHeader_2.54mm:PinHeader_2x01_P2.54mm_Vertical, symbol Jumper:Jumper_2_Open
- removed JP4: JP4, Connector_PinHeader_2.54mm:PinHeader_2x01_P2.54mm_Vertical, symbol Jumper:Jumper_2_Open
- removed Q1, Q2: BSS138, Package_TO_SOT_SMD:SOT-23, symbol Transistor_FET:BSS138
- removed R2, R3, R5, R6, R7, R8: 4.7K, Resistor_SMD:R_0603_1608Metric, symbol Device:R
- removed R4, R9: 10K, Resistor_SMD:R_0603_1608Metric, symbol Device:R
- removed U1: MCP4728, Package_SO:MSOP-10_3x3mm_P0.5mm, symbol Analog_DAC:MCP4728
- removed U2: ATmega328PB-AU, Package_QFP:TQFP-32_7x7mm_P0.8mm, symbol MCU_Microchip_ATmega:ATmega328PB-A
- removed Y1: 16MHz, Crystal:Crystal_HC49-4H_Vertical, symbol Device:Crystal
- added J3: AUX_ALT, Connector_PinHeader_2.54mm:PinHeader_2x04_P2.54mm_Vertical, symbol Connector_Generic:Conn_02x04_Odd_Even
- added J4: ESPFlash, Connector_IDC:IDC-Header_2x03_P2.54mm_Vertical, symbol Connector_Generic:Conn_02x03_Odd_Even
- added J5: FRONT_PANEL, Connector_PinHeader_2.54mm:PinHeader_2x08_P2.54mm_Vertical, symbol Connector_Generic:Conn_02x08_Odd_Even
- added J6: DISPLAY, Connector_PinHeader_2.54mm:PinHeader_1x10_P2.54mm_Vertical, symbol Connector_Generic:Conn_01x10
- added U1: ESP32-WROOM-32D, RF_Module:ESP32-WROOM-32, symbol RF_Module:ESP32-WROOM-32D
- C1: value 100nF -> 10uF; LCSC C1591 -> C2922482; MOUSER 187-CL10B104KB8NNNC -> 187-CL10A106MA8NRNC; MPN CL10B104KB8NNNC -> CL10A106MA8NRNC
- C2: value 10uF -> 100nF; LCSC C2922482 -> C1591; MOUSER 187-CL10A106MA8NRNC -> 187-CL10B104KB8NNNC; MPN CL10A106MA8NRNC -> CL10B104KB8NNNC
- J1: renamed from J3; value MIC -> AUX1
- J2: renamed from J4; value LINE IN -> AUX2
- R1: value 1K -> 10K; LCSC C22548 -> C98220; MOUSER 603-RC0603FR-071KL -> 603-RC0603FR-0710KL; MPN RC0603FR-071KL -> RC0603FR-0710KL
- renumbered H12 to H1, H3 to H10, H2 to H11, H1 to H12, H10 to H2, H8 to H3, H6 to H4, H11 to H5, H9 to H6, H5 to H8, H4 to H9, J9 to J7
Connections:
- net RESET is gone; now on net +3V3: C1.1
- net +3V3: now also C2.1, J7.2 (+3.3V), J4.2 (Pin_2), J5.3 (Pin_3), J6.2 (Pin_2), U1.2 (VDD); no longer J7.1 (+3.3V)
- net +5V: now also J5.5 (Pin_5); no longer C2.1
- net GND: now also C1.2, J7.1 (GND), R1.2, J4.4 (Pin_4), J5.1 (Pin_1), J6.1 (Pin_1), U1.1 (GND), U1.15 (GND), U1.38 (GND), U1.39 (GND); no longer J7.2 (GND)
- net MISO: now also J6.9 (Pin_9), U1.31 (IO19)
- net MOSI: now also J6.7 (Pin_7), U1.37 (IO23)
- net RXD: now also J4.5 (Pin_5), U1.34 (RXD0/IO3)
- net SCK: now also J6.8 (Pin_8), U1.30 (IO18); no longer R1.1
- net TXD: now also J4.3 (Pin_3), U1.35 (TXD0/IO1)
- net AUX2TN: now reaches J2.TN
- net AUX2TN: now also J3.2 (Pin_2)
- net AUX2S: now reaches J2.S, J7.10 (AUX2S)
- net AUX2S: now also J3.4 (Pin_4), J3.6 (Pin_6)
- net AUX2RN: now reaches J2.RN
- net AUX2RN: now also J3.8 (Pin_8)
- net AUX1S: now reaches J1.S, J7.7 (AUX1S)
- net AUX1S: now also J3.3 (Pin_3), J3.5 (Pin_5)
- net AUX1TN: now reaches J1.TN
- net AUX1TN: now also J3.1 (Pin_1)
- net at J1.R: now also J7.8 (AUX1R)
- net AUX1RN: now reaches J1.RN
- net AUX1RN: now also J3.7 (Pin_7)
- net at J1.T: now also J7.9 (AUX1T); no longer J7.6 (MIC_IN_T)
- net at J2.T: now also J7.12 (AUX2T); no longer J7.8 (LINE_IN_T)
- net at J2.R: now also J7.11 (AUX2R); no longer J7.9 (LINE_IN_R)
- net LINE_LEFT renamed AUX1R
- net AUX1R: now also U1.9 (IO33)
- net LINE_RIGHT renamed AUX2T
- net AUX2T: now also U1.10 (IO25)
- net MIC renamed AUX1T
- net AUX1T: now also U1.8 (IO32)
- new net AUX2R: J7.6 (A2R), U1.11 (IO26)
- new net BUZZER: J5.15 (Pin_15), U1.14 (IO12)
- new net CARD_CS: J6.5 (Pin_5), U1.16 (IO13)
- new net CIO1: J5.10 (Pin_10)
- new net CIO2: J5.12 (Pin_12)
- new net CIO3: J5.14 (Pin_14)
- new net CS: U1.29 (IO5)
- new net EN: J4.1 (Pin_1), U1.3 (EN)
- new net ENC_A: J5.7 (Pin_7), U1.36 (IO22)
- new net ENC_B: J5.9 (Pin_9), U1.33 (IO21)
- new net ENC_SW: J5.11 (Pin_11), U1.28 (IO17)
- new net IO0: J4.6 (Pin_6), U1.25 (IO0)
- new net IO2: R1.1, U1.24 (IO2)
- new net LCD_CS: J6.6 (Pin_6), U1.27 (IO16)
- new net LCD_DC: J6.4 (Pin_4), U1.13 (IO14)
- new net LCD_LITE: J6.10 (Pin_10), U1.12 (IO27)
- new net LCD_RST: J6.3 (Pin_3), U1.23 (IO15)
- new net LED_DATA: J5.13 (Pin_13), U1.26 (IO4)
- new net LVL_1: J5.2 (Pin_2), U1.4 (SENSOR_VP)
- new net LVL_2: J5.4 (Pin_4), U1.5 (SENSOR_VN)
- new net LVL_3: J5.6 (Pin_6), U1.6 (IO34)
- new net LVL_4: J5.8 (Pin_8), U1.7 (IO35)
- no-connect marks 12 -> 7
Other:
- sheet PSU renamed Power Supply
- added sheet Output (output.kicad_sch)
- sheet Power Supply ports: added none; removed VBAT, VIN
- note added: "Adafruit 1.8" Color TFT (ADA358) & SD card reader"
- note added: "Aux Input/Output"
- note added: "Aux Module e.g. audio module, trigger module, etc"
- note added: "Boot Strapping Pins: IO 0,2,5,12,15"
- note added: "CIO1, CIO2, CIO3 are GPIOs from the CO-MCU (Pico) Pin 16 is for polarity protection"
- note added: "ESP-PROG"
- note removed: "3.3V logic"
- note removed: "Audio Input"
- note removed: "Audio Module"
- note removed: "DAC"
- note removed: "I^{2}C Level Shifter / Pull-ups"
- note removed: "MCU"
- note removed: "Output Channels"
- note removed: "max 400kHz I2C min 130us/ch set time addr = 0x60"
- moved on the sheet: H1, H10, H11, H12, H2, H3, H4, H5, H6, H7, H8, H9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
