File: hardware/pcb/main_board/SW-324.kicad_pcb (KiCad board)
At the start: 2 copper layers, 177.8 x 119.4 mm, 97 parts, among them J1 AUX1, J10 SERIAL, J11 DEBUG, J12 Channel 1, J13 Channel 2, J14 Channel 3, J15 Channel 4, J16 CH_1, J17 CH_2, J18 CH_3, J19 CH_4, J2 AUX2, J3 AUX_ALT, J4 ESPFlash, J5 FRONT_PANEL, J6 DISPLAY, J7 locked, J8 PWR, J9 BAT, Q1 DMG2301L-7, SW1 PWR_SW, U1 ESP32-WROOM-32D, U2 TPS5430DDA, U3 TPS5430DDA, U4 LM2941, U5 NCP1117-3.3, U6 Pico, U7 MCP4728, U8 ADS1015

Commit message: fix comments
Parts:
- removed the C1 at (103.3, 89.2)
- removed the C2 at (100.6, 89.2)
- removed the J1 at (139.7, 146.1)
- removed the J2 at (154.9, 146.1)
- removed the J3 at (122.2, 139.0)
- removed the J4 at (94.0, 104.1)
- removed the J5 at (94.0, 77.5)
- removed the J6 at (103.5, 113.0)
- removed the J7 at (113.0, 125.7)
- removed the R1 at (119.8, 109.5)
- removed the U1 at (114.9, 96.7)
- added C18: 10uF, Capacitor_SMD:C_0603_1608Metric, F.Cu at (101.6, 88.9)
- added C19: 100nF, Capacitor_SMD:C_0603_1608Metric, F.Cu at (103.5, 88.9)
- added D5: Diode, Diode_SMD:D_SOD-123F, F.Cu at (0.81, 118.8)
- added J13: AUX1, SaawLib:STX-3100-5N, F.Cu at (139.7, 146.1)
- added J14: AUX2, SaawLib:STX-3100-5N, F.Cu at (154.9, 146.1)
- added J15: AUX_ALT, Connector_PinHeader_2.54mm:PinHeader_2x04_P2.54mm_Vertical, F.Cu at (122.2, 139.0)
- added J16: ESPFlash, Connector_IDC:IDC-Header_2x03_P2.54mm_Vertical, F.Cu at (94.0, 104.1)
- added J17: FRONT_PANEL, Connector_IDC:IDC-Header_2x04_P2.54mm_Vertical, F.Cu at (94.0, 83.2)
- added J18: DISPLAY, Connector_PinHeader_2.54mm:PinHeader_1x10_P2.54mm_Vertical, F.Cu at (103.5, 113.0)
- added J19: SW-32MA, SaawLib:SW-32MA_Socket, F.Cu at (113.0, 125.7)
- added JP1: USB_PWR, Jumper:SolderJumper-2_P1.3mm_Bridged_RoundedPad1.0x1.5mm, F.Cu at (0.22, 122.2)
- added JP2: CO_BOOT, Connector_PinHeader_2.54mm:PinHeader_1x02_P2.54mm_Vertical, F.Cu at (133.3, 95.2)
- added R17: 10K, Resistor_SMD:R_0603_1608Metric, F.Cu at (23.1, 110.5)
- added R18: 10K, Resistor_SMD:R_0603_1608Metric, F.Cu at (18.4, 118.2)
- added R19: 10K, Resistor_SMD:R_0603_1608Metric, F.Cu at (14.4, 118.2)
- added R20: 10K, Resistor_SMD:R_0603_1608Metric, F.Cu at (19.1, 110.5)
- added R21: 10K, Resistor_SMD:R_0603_1608Metric, F.Cu at (19.1, 115.6)
- added R22: 10K, Resistor_SMD:R_0603_1608Metric, F.Cu at (31.0, 108.0)
- added U8: ESP32-WROOM-32D, RF_Module:ESP32-WROOM-32, F.Cu at (114.9, 96.7)
- J3: renamed from J10; footprint Connector_PinHeader_2.54mm:PinHeader_1x06_P2.54mm_Vertical -> Connector_PinHeader_2.54mm:PinHeader_1x04_P2.54mm_Vertical
- J4: renamed from J11; value DEBUG -> SWD; footprint Connector_PinHeader_2.54mm:PinHeader_1x03_P2.54mm_Vertical -> Connector_PinHeader_2.54mm:PinHeader_1x05_P2.54mm_Vertical
- moved J3 3.81 mm to (133.3, 78.7)
- moved TP6 1.98 mm to (88.3, 85.7)
- renumbered C3 to C1, C12 to C10, C13 to C11, C14 to C12, C15 to C13, C16 to C14, C17 to C15, C18 to C16, C19 to C17, C4 to C2, C6 to C4, C8 to C6, C9 to C7, C10 to C8, C11 to C9, D5 to D6, D6 to D7, J8 to J1, J17 to J10, J18 to J11, J19 to J12, J9 to J2, J12 to J5, J13 to J6, J14 to J7, J15 to J8, J16 to J9, JP1 to JP3, JP2 to JP4, JP3 to JP5, JP4 to JP6, R2 to R1, R11 to R10, R12 to R11, R13 to R12, R14 to R13, R15 to R14, R16 to R15, R17 to R16, R3 to R2, R4 to R3, R5 to R4, R6 to R5, R7 to R6, R8 to R7, R9 to R8, R10 to R9, U2 to U1, U3 to U2, U4 to U3, U5 to U4, U6 to U5, U7 to U6, U8 to U7
Connections:
- net /Output/CH1_LVL renamed /Controller/CH1_LVL
- net /Output/CH1_SENSE renamed /Controller/CH1_SENSE
- net /Output/CH2_LVL renamed /Controller/CH2_LVL
- net /Output/CH2_SENSE renamed /Controller/CH2_SENSE
- net /Output/CH3_LVL renamed /Controller/CH3_LVL
- net /Output/CH3_SENSE renamed /Controller/CH3_SENSE
- net /Output/CH4_LVL renamed /Controller/CH4_LVL
- net /Output/CH4_SENSE renamed /Controller/CH4_SENSE
- net Net-(Q1-Pad1) renamed VBUS
- J3 pad 2: unconnected-(J10-Pad2) -> +3V3
- J3 pad 3: unconnected-(J10-Pad3) -> /Controller/RXD0
- J3 pad 4: /Output/RXD -> /Controller/TXD0
- J4 pad 1: /Output/SWCLK -> GND
- J4 pad 2: GND -> +3V3
- J4 pad 3: /Output/SWDIO -> /Controller/SWCLK
- J5 pad 6: /Output/CH1_PA -> /Controller/CH1_PA
- J5 pad 7: /Output/CH1_PB -> /Controller/CH1_PB
- J6 pad 6: /Output/CH2_PA -> /Controller/CH2_PA
- J6 pad 7: /Output/CH2_PB -> /Controller/CH2_PB
- J7 pad 6: /Output/CH3_PA -> /Controller/CH3_PA
- J7 pad 7: /Output/CH3_PB -> /Controller/CH3_PB
- J8 pad 6: /Output/CH4_PA -> /Controller/CH4_PA
- J8 pad 7: /Output/CH4_PB -> /Controller/CH4_PB
- R1 pad 1: /REG_EN -> /Controller/REG_EN
- R10 pad 2: /VBAT_SENSE -> /Controller/VBAT_SENSE
- R11 pad 1: /VBAT_SENSE -> /Controller/VBAT_SENSE
- R13 pad 2: /Output/SCL_PER -> /Controller/SCL_PER
- R14 pad 2: /Output/SDA_PER -> /Controller/SDA_PER
- R15 pad 2: /Output/~{LDAC} -> /Controller/~{LDAC}
- R16 pad 1: /Output/RDY -> /Controller/~{RDY}
- U1 pad 5: /REG_EN -> /Controller/REG_EN
- U5 pad 1: /Output/TXD -> /Controller/TXD0
- U5 pad 10: /Output/CH4_PB -> /Controller/CH3_PA
- U5 pad 11: /Output/CH3_PA -> /Controller/CH3_PB
- U5 pad 12: /Output/CH3_PB -> /Controller/CH4_PA
- U5 pad 14: /Output/CH2_PA -> /Controller/CH4_PB
- U5 pad 15: /Output/CH2_PB -> /Controller/CH1_PA
- U5 pad 16: /Output/CH1_PA -> /Controller/CH1_PB
- U5 pad 17: /Output/CH1_PB -> /Controller/CH2_PA
- U5 pad 19: /Output/SDA_PER -> /Controller/CH2_PB
- U5 pad 2: /Output/RXD -> /Controller/RXD0
- U5 pad 20: /Output/SCL_PER -> /Comms Controller/~{BOOT/INT}
- U5 pad 21: /MOSI -> /Comms Controller/MOSI
- U5 pad 22: /CS -> /Comms Controller/~{CS}
- U5 pad 24: /SCK -> /Comms Controller/SLK
- U5 pad 25: /MISO -> /Comms Controller/MISO
- U5 pad 26: /Output/RDY -> /Comms Controller/SD
- U5 pad 27: /Output/~{LDAC} -> /Comms Controller/WS
- U5 pad 29: /CIO1 -> /Comms Controller/SCK
- U5 pad 30: unconnected-(U6-Pad30) -> /Controller/~{RST}
- U5 pad 31: /VBAT_SENSE -> /Controller/~{RDY}
- U5 pad 32: /CIO2 -> /Controller/~{LDAC}
- U5 pad 34: /CIO3 -> /Controller/VBAT_SENSE
- U5 pad 4: /REG_EN -> /Controller/SDA_PER
- U5 pad 41: /Output/SWCLK -> /Controller/SWCLK
- U5 pad 43: /Output/SWDIO -> /Controller/SWD
- U5 pad 5: unconnected-(U6-Pad5) (its old number) -> /Controller/SCL_PER
- U5 pad 6: unconnected-(U6-Pad6) -> /Comms Controller/RXD
- U5 pad 7: unconnected-(U6-Pad7) -> /Comms Controller/TXD
- U5 pad 9: /Output/CH4_PA -> /Controller/REG_EN
- U6 pad 2: /Output/SCL_PER -> /Controller/SCL_PER
- U6 pad 3: /Output/SDA_PER -> /Controller/SDA_PER
- U6 pad 4: /Output/~{LDAC} -> /Controller/~{LDAC}
- U7 pad 10: /Output/SCL_PER -> /Controller/SCL_PER
- U7 pad 2: /Output/RDY -> /Controller/~{RDY}
- U7 pad 9: /Output/SDA_PER -> /Controller/SDA_PER
Routing:
- net /CIO3: track 164.9 -> 0.00 mm, vias 3 -> 0
- net /CIO2: track 159.4 -> 0.00 mm, vias 3 -> 0
- net /CIO1: track 152.8 -> 0.00 mm, vias 1 -> 0
- net /MOSI: track 123.9 -> 0.00 mm, vias 1 -> 0
- net /Comms Controller/MOSI: track 0.00 -> 117.7 mm, vias 0 -> 1
- net /Output/TXD: track 117.5 -> 0.00 mm
- net /Output/RXD: track 115.5 -> 0.00 mm
- net /SCK: track 107.3 -> 0.00 mm, vias 1 -> 0
- net /CS: track 105.9 -> 0.00 mm, vias 2 -> 0
- net /MISO: track 105.2 -> 0.00 mm
- net /Comms Controller/SCK: track 0.00 -> 103.4 mm, vias 0 -> 1
- net /Comms Controller/~{CS}: track 0.00 -> 100.0 mm, vias 0 -> 2
- net /Comms Controller/MISO: track 0.00 -> 99.4 mm
- net /Controller/TXD0: track 0.00 -> 95.9 mm
- net /Controller/RXD0: track 0.00 -> 92.9 mm
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