File: hardware/pcb/main_board/SW-324.kicad_sch (KiCad schematic)
At the start: 23 parts, among them J1 AUX1, J2 AUX2, J3 AUX_ALT, J4 ESPFlash, J5 FRONT_PANEL, J6 DISPLAY, J7 SW-32MA, U1 ESP32-WROOM-32D

Commit message: fix comments
Parts:
- removed C1: 10uF, Capacitor_SMD:C_0603_1608Metric, symbol Device:C_Small
- removed C2: 100nF, Capacitor_SMD:C_0603_1608Metric, symbol Device:C_Small
- removed J1: AUX1, SaawLib:STX-3100-5N, symbol Connector:AudioJack3_SwitchTR
- removed J2: AUX2, SaawLib:STX-3100-5N, symbol Connector:AudioJack3_SwitchTR
- removed J3: AUX_ALT, Connector_PinHeader_2.54mm:PinHeader_2x04_P2.54mm_Vertical, symbol Connector_Generic:Conn_02x04_Odd_Even
- removed J4: ESPFlash, Connector_IDC:IDC-Header_2x03_P2.54mm_Vertical, symbol Connector_Generic:Conn_02x03_Odd_Even
- removed J5: FRONT_PANEL, Connector_PinHeader_2.54mm:PinHeader_2x08_P2.54mm_Vertical, symbol Connector_Generic:Conn_02x08_Odd_Even
- removed J6: DISPLAY, Connector_PinHeader_2.54mm:PinHeader_1x10_P2.54mm_Vertical, symbol Connector_Generic:Conn_01x10
- removed J7: SW-32MA, SaawLib:SW-32MA_Socket, symbol SaawLib:SW-32MA
- removed R1: 10K, Resistor_SMD:R_0603_1608Metric, symbol Device:R
- removed U1: ESP32-WROOM-32D, RF_Module:ESP32-WROOM-32, symbol RF_Module:ESP32-WROOM-32D
Connections:
- no-connect marks 7 -> 0
Other:
- sheet Output renamed Controller
- added sheet Comms Controller (comms.kicad_sch)
- sheet Controller ports: added RXD1, SD, SLK, TXD1, VBAT_SENSE, WS, ~{CO_BOOT/INT}; removed IO22, IO27, IO28, VBAT
- note added: "--> I2S -->"
- note added: "High-level controller responsible for wireless comms, display, and user controls"
- note added: "Low-level controller responsible for controlling output module drivers and routine generation"
- note added: "MASTER <--> SPI <--> SLAVE"
- note added: "Provides power (+9V, +5V, and +3.3V) and battery charging."
- note added: "Serial (Reprogramming)"
- note removed: "Adafruit 1.8" Color TFT (ADA358) & SD card reader"
- note removed: "Aux Input/Output"
- note removed: "Aux Module e.g. audio module, trigger module, etc"
- note removed: "Boot Strapping Pins: IO 0,2,5,12,15"
- note removed: "CIO1, CIO2, CIO3 are GPIOs from the CO-MCU (Pico) Pin 16 is for polarity protection"
- note removed: "ESP-PROG"
- note removed: "Power Supply / Charger"
- note removed: "REG_EN enables the 9V reg used by output modules."
- title: SW-3240: Main Board -> SW-324: Main Board
