File: hardware/pcb/main_board/output.kicad_sch (KiCad schematic)
At the start: 25 parts, among them J10 SERIAL, J11 DEBUG, J12 Channel 1, J13 Channel 2, J14 Channel 3, J15 Channel 4, J16 CH_1, J17 CH_2, J18 CH_3, J19 CH_4, Q1 DMG2301L-7, U6 Pico, U7 MCP4728, U8 ADS1015

Commit message: fix comments
Parts:
- added JP2: CO_BOOT, Connector_PinHeader_2.54mm:PinHeader_1x02_P2.54mm_Vertical, symbol Jumper:Jumper_2_Open
- J3: renamed from J10; footprint Connector_PinHeader_2.54mm:PinHeader_1x06_P2.54mm_Vertical -> Connector_PinHeader_2.54mm:PinHeader_1x04_P2.54mm_Vertical; symbol Connector_Generic:Conn_01x06 -> Connector_Generic:Conn_01x04; now in the parts list
- J4: renamed from J11; value DEBUG -> SWD; footprint Connector_PinHeader_2.54mm:PinHeader_1x03_P2.54mm_Vertical -> Connector_PinHeader_2.54mm:PinHeader_1x05_P2.54mm_Vertical; symbol Connector_Generic:Conn_01x03 -> Connector_Generic:Conn_01x05; now in the parts list
- renumbered C17 to C15, C18 to C16, C19 to C17, J17 to J10, J18 to J11, J19 to J12, J12 to J5, J13 to J6, J14 to J7, J15 to J8, J16 to J9, JP1 to JP3, JP2 to JP4, JP3 to JP5, JP4 to JP6, R14 to R13, R15 to R14, R16 to R15, R17 to R16, U6 to U5, U7 to U6, U8 to U7
Connections:
- net IO27 is gone; now on net ~{LDAC}: U5.32 (GPIO27_ADC1)
- net VBAT is gone; now on net ~{RDY}: U5.31 (GPIO26_ADC0)
- net +3V3: now also J3.2 (Pin_2), J4.2 (Pin_2)
- net CH1_PA: now also U5.15 (GPIO11); no longer U5.16 (GPIO12)
- net CH1_PB: now also U5.16 (GPIO12); no longer U5.17 (GPIO13)
- net CH2_PA: now also U5.17 (GPIO13); no longer U5.14 (GPIO10)
- net CH2_PB: now also U5.19 (GPIO14); no longer U5.15 (GPIO11)
- net CH3_PA: now also U5.10 (GPIO7); no longer U5.11 (GPIO8)
- net CH3_PB: now also U5.11 (GPIO8); no longer U5.12 (GPIO9)
- net CH4_PA: now also U5.12 (GPIO9); no longer U5.9 (GPIO6)
- net CH4_PB: now also U5.14 (GPIO10); no longer U5.10 (GPIO7)
- net GND: now also J4.1 (Pin_1), JP2.2 (B); no longer J4.2 (Pin_2)
- net REG_EN: now also U5.9 (GPIO6); no longer U5.4 (GPIO2)
- net SCL_PER: now also U5.5 (GPIO3); no longer U5.20 (GPIO15)
- net SDA_PER: now also U5.4 (GPIO2); no longer U5.19 (GPIO14)
- net SWCLK: now also J4.3 (Pin_3); no longer J4.1 (Pin_1)
- net ~{LDAC}: no longer U5.27 (GPIO21)
- net ~{RST}: now reaches U5.30 (RUN)
- net ~{RST}: now also J4.5 (Pin_5)
- net VBUS: now reaches Q1.1 (G), U5.40 (VBUS)
- net TXD1: now reaches U5.6 (GPIO4)
- net RXD1: now reaches U5.7 (GPIO5)
- net RXD0: now reaches J3.3 (Pin_3)
- net RXD0: now also U5.2 (GPIO1)
- net IO22 renamed SLK
- net IO28 renamed VBAT_SENSE
- net RDY renamed ~{RDY}
- net ~{RDY}: no longer U5.26 (GPIO20)
- net RXD renamed TXD0
- net TXD0: now also U5.1 (GPIO0); no longer U5.2 (GPIO1)
- net SWDIO renamed SWD
- net SWD: now also J4.4 (Pin_4); no longer J4.3 (Pin_3)
- removed net TXD: J3.5 (Pin_5), U5.1 (GPIO0)
- new net SD: U5.26 (GPIO20)
- new net WS: U5.27 (GPIO21)
- new net ~{CO_BOOT/INT}: JP2.1 (A), U5.20 (GPIO15)
- no-connect marks 20 -> 13
Other:
- note added: "Comms Controller Serial Bootloader (IO0) & UART Passthrough"
- title: SW-3240: Main Board - Output -> SW-324: Main Board - Controller
