File: hardware/pcb/main_board/power.kicad_sch (KiCad schematic)
At the start: 49 parts, among them SW1 PWR_SW, U3 TPS5430DDA, U4 TPS5430DDA, U5 LM2941, U6 NCP1117-3.3

Commit message: refactor
Other:
- title: SW-3240: Power Supply -> SW-3240: Main Board - Power Supply
Changed lines of the file:
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@@
   (paper "A4")
   (title_block
-    (title "SW-3240: Power Supply")
+    (title "SW-3240: Main Board - Power Supply")
     (date "2022-04-07")
     (rev "1")

Commit message: update part numbers
Parts:
- removed C20: 330uF, Capacitor_THT:C_Radial_D8.0mm_H11.5mm_P3.50mm, symbol Device:C_Polarized
- C17, C8, C9: footprint Capacitor_THT:C_Radial_D8.0mm_H11.5mm_P3.50mm -> Capacitor_THT:CP_Radial_D6.3mm_P2.50mm; LCSC (none) -> C1579509; MOUSER (none) -> 667-EEU-FM1E101; MPN (none) -> EEU-FM1E101
- renumbered C21 to C20, C22 to C21, C23 to C22, TP2 to TP1, TP3 to TP2, TP4 to TP3, TP5 to TP4, TP6 to TP5, TP7 to TP6
Other:
- note added: "ESR: 100 mΩ - 1 Ω"
- note removed: "ESR 0.1 to 1.0R"
- note removed: "TODO: Check charger caps values / footprints Check regulator bulk caps footprints"

Commit message: redesign
Parts:
- removed C22: 100nF, Capacitor_SMD:C_0603_1608Metric, symbol Device:C
- removed R20: 1K, Resistor_SMD:R_0603_1608Metric, symbol Device:R
- added J8: PWR, SaawLib:BarrelJack_CUI_PJ-102AH_Horizontal, symbol Connector:Barrel_Jack_Switch
- added J9: BAT, Connector_JST:JST_XH_B2B-XH-A_1x02_P2.50mm_Vertical, symbol Connector:Screw_Terminal_01x02
- added R10: 10K, Resistor_SMD:R_0603_1608Metric, symbol Device:R
- R13: renamed from R21; value 1K -> 1.5K; LCSC C22548 -> C114668; MOUSER 603-RC0603FR-071KL -> 603-RC0603FR-071K5L; MPN RC0603FR-071KL -> RC0603FR-071K5L
- renumbered C15 to C10, C16 to C11, C17 to C12, C18 to C13, C19 to C14, C20 to C15, C21 to C16, C8 to C3, C9 to C4, C10 to C5, C11 to C6, C12 to C7, C13 to C8, C14 to C9, D2 to D1, D3 to D2, D4 to D3, D5 to D4, D6 to D5, D7 to D6, R18 to R11, R19 to R12, R10 to R2, R11 to R3, R12 to R4, R13 to R5, R14 to R6, R15 to R7, R16 to R8, R17 to R9, U3 to U2, U4 to U3, U5 to U4, U6 to U5
Connections:
- net +12V: now also R10.1; no longer R11.1
- net +9V: now also R13.2
- net GND: now also J8.2, J9.2 (Pin_2)
- net VBAT: no longer names the net of F2.2
- net VBAT: now also J9.1 (Pin_1)
- net VIN: no longer names the net of D1.2 (A)
- net VIN: now also J8.1
- new net: R10.2, R11.1
- no-connect marks 5 -> 6
Other:
- note removed: "Vf: ~2.1V"
- note removed: "Vf: ~3.6V"
- moved on the sheet: C9, D1, D5, D6, F2, R11, R12, R13, R9

Commit message: fix comments
Parts:
- added D5: Diode, Diode_SMD:D_SOD-123F, symbol Device:D_Schottky
- added JP1: USB_PWR, Jumper:SolderJumper-2_P1.3mm_Bridged_RoundedPad1.0x1.5mm, symbol Jumper:SolderJumper_2_Bridged
- renumbered C3 to C1, C12 to C10, C13 to C11, C14 to C12, C15 to C13, C16 to C14, C4 to C2, C5 to C3, C6 to C4, C7 to C5, C8 to C6, C9 to C7, C10 to C8, C11 to C9, D5 to D6, D6 to D7, J8 to J1, J9 to J2, R2 to R1, R11 to R10, R12 to R11, R13 to R12, R3 to R2, R4 to R3, R5 to R4, R6 to R5, R7 to R6, R8 to R7, R9 to R8, R10 to R9, U2 to U1, U3 to U2, U4 to U3, U5 to U4
Connections:
- net +5V: now also D5.1 (K)
- new net: D5.2 (A), JP1.2 (B)
- new net VBUS: JP1.1 (A)
Other:
- note added: "Alt Basic Part: AMS1117-3.3 ??"
- title: SW-3240: Main Board - Power Supply -> SW-324: Main Board - Power Supply
