File: hardware/pcb/modules/output/SW-32MO11/SW-32MO11.kicad_pcb (KiCad board)
At the start: 2 copper layers, 65 x 24.6 mm, 23 parts, among them Q1 IRF9Z24NPBF, Q2 DMG3404L-7, Q3 DMG3404L-7, T1 42TL004-RC, U1 SW-32MO, U2 LM358ADT/TLV272IS-13

Commit message: redesign
Parts:
- Q1: value IRF9Z24NPBF -> IRFR9024NTRPBF; footprint Package_TO_SOT_THT:TO-220-3_Horizontal_TabDown -> Package_TO_SOT_SMD:TO-252-3_TabPin2
- moved Q1 11.4 mm to (116.7, 74.7), turned to 0 degrees
- moved R3 6.22 mm to (108.6, 74.9)
Routing:
- net /PULSE_SRC: track 43.9 -> 34.1 mm
- net +9V: track 11.1 -> 8.47 mm
- net Net-(Q1-Pad1): track 18.0 -> 19.8 mm, vias 1 -> 2
Other:
- board text added: "SW-32MO11"
- board text removed: "SW-32MO10"
