File: hardware/pcb/modules/output/SW-32MO11/SW-32MO11.kicad_sch (KiCad schematic)
At the start: 23 parts, among them Q1 IRF9Z24NPBF, Q2 DMG3404L-7, Q3 DMG3404L-7, T1 42TL004-RC, U1 SW-32MO, U2 LM358ADT/TLV272IS-13

Commit message: redesign
Parts:
- Q1: value IRF9Z24NPBF -> IRFR9024NTRPBF; footprint Package_TO_SOT_THT:TO-220-3_Horizontal_TabDown -> Package_TO_SOT_SMD:TO-252-3_TabPin2; MPN IRF9Z24NPBF -> IRFR9024NTRPBF
Other:
- title: SW-32MO10 -> SW-32MO11
Changed lines of the file:
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@@
   (paper "A4")
   (title_block
-    (title "SW-32MO10")
-    (date "2022-05-05")
+    (title "SW-32MO11")
+    (date "2022-06-10")
     (rev "1")
     (company "saawsm")
@@
     (in_bom yes) (on_board yes)
     (property "Reference" "Q1" (id 0) (at 130.81 25.4 90))
-    (property "Value" "IRF9Z24NPBF" (id 1) (at 130.81 27.94 90))
-    (property "Footprint" "Package_TO_SOT_THT:TO-220-3_Horizontal_TabDown" (id 2) (at 133.35 29.21 0)
+    (property "Value" "IRFR9024NTRPBF" (id 1) (at 130.81 27.94 90))
+    (property "Footprint" "Package_TO_SOT_SMD:TO-252-3_TabPin2" (id 2) (at 133.35 29.21 0)
       (effects (font (size 1.27 1.27)) hide)
     )
@@
       (effects (font (size 1.27 1.27)) hide)
     )
-    (property "MPN" "IRF9Z24NPBF" (id 4) (at 130.81 34.29 0)
+    (property "MPN" "IRFR9024NTRPBF" (id 4) (at 130.81 34.29 0)
       (effects (font (size 1.27 1.27)) hide)
     )
@@
     )
     (path "/0ff57116-dd3c-413e-b372-227f3cd30a98"
-      (reference "Q1") (unit 1) (value "IRF9Z24NPBF") (footprint "Package_TO_SOT_THT:TO-220-3_Horizontal_TabDown")
+      (reference "Q1") (unit 1) (value "IRFR9024NTRPBF") (footprint "Package_TO_SOT_SMD:TO-252-3_TabPin2")
     )
     (path "/32e1aed6-e06d-402f-b13b-cddeae58cd61"
