File: hardware/pcb/modules/auxiliary/audio/SW-32MA1/SW-32MA1.kicad_sch (KiCad schematic)
At the start: 24 parts, among them U1 Opamp_Quad, U2 SW-32MA

Commit message: redesign
Parts:
- R16: now left out of the parts list
- R4, R5, R6, R7, R8, R9: value 10K -> 100K
Connections:
- net +3V3: now also U2.2 (+3.3V); no longer U2.1 (+3.3V)
- net GND: now also U2.1 (GND); no longer U2.2 (GND)
- net LINE_IN_R: now also U2.11 (AUX2R); no longer U2.9 (LINE_IN_R)
- net LINE_IN_T: now also U2.12 (AUX2T); no longer U2.8 (LINE_IN_T)
- net LINE_LEFT: now also U2.5 (A2T); no longer U2.4 (LINE_LEFT)
- net LINE_RIGHT: now also U2.6 (A2R); no longer U2.5 (LINE_RIGHT)
- net MIC_IN: now also U2.9 (AUX1T); no longer U2.6 (MIC_IN_T)
- no-connect marks 0 -> 2
