File: kicad/SW3F1 - Front Panel/SW3F1 - Front Panel.kicad_pcb (KiCad board)
At the start: 2 copper layers, 137.2 x 45.7 mm, 50 parts, among them J1 MAIN_BOARD, J2 LED_OUT, Q1 DMG2301L-7, SW1 PEC11R-42xxK-S0024, SW2 BTN1, SW3 BTN2, SW4 BTN3, SW5 BTN4, U1 PCF8574, U2 PCF8591

Commit message: misc. cleanup
Parts:
- moved H5 2.54 mm to (143.5, 105.4)
- moved J1 0.10 mm to (117.6, 95.5)

Commit message: add optional I2C pullups
Parts:
- added JP1: SolderJumper_2_Open, Jumper:SolderJumper-2_P1.3mm_Open_RoundedPad1.0x1.5mm, B.Cu at (165.1, 111.8)
- added JP2: SolderJumper_2_Open, Jumper:SolderJumper-2_P1.3mm_Open_RoundedPad1.0x1.5mm, B.Cu at (161.3, 111.8)
- added R4: 10K, Resistor_SMD:R_0603_1608Metric, B.Cu at (165.1, 116.2)
- added R6: 10K, Resistor_SMD:R_0603_1608Metric, B.Cu at (161.3, 116.2)
- renumbered R8 to R10, R9 to R11, R10 to R12, R4 to R5, R5 to R7, R7 to R9
Routing:
- net +3.3V: track 278.1 -> 296.5 mm
- net /SCL: track 96.4 -> 106.1 mm
- net Net-(JP2-Pad2): track 0.00 -> 2.99 mm
- net Net-(JP1-Pad2): track 0.00 -> 2.99 mm
- net /SDA: track 99.2 -> 101.4 mm

Commit message: update MPN for rotary encoder
Parts:
- SW1: value PEC11R-42xxK-S0024 -> PEC11R-4215K-S0024
Changed lines of the file:
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@@
   (footprint "SaawLib:Rotary_Encoder_Switched_PEC11R" locked (layer "F.Cu")
     (at 130.81 92.71)
-    (property "MPN" "PEC11R-42xxK-S0024")
+    (property "MPN" "PEC11R-4215K-S0024")
     (property "Sheetfile" "SW3F1 - Front Panel.kicad_sch")
     (property "Sheetname" "")
@@
       (effects (font (size 1 1) (thickness 0.15)))
     )
-    (fp_text value "PEC11R-42xxK-S0024" (at 5.125 9.725) (layer "F.Fab")
+    (fp_text value "PEC11R-4215K-S0024" (at 5.125 9.725) (layer "F.Fab")
       (effects (font (size 1 1) (thickness 0.15)))
     )

Commit message: simplify bom - use SS24FL
Parts:
- D1: value MBR120 -> SS24FL
Changed lines of the file:
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@@
   (title_block
     (title "SW3F1 - Front Panel")
-    (date "2022-11-05")
+    (date "2022-12-21")
     (rev "1")
     (company "saawsm")
@@
     (descr "D_SOD-123F")
     (tags "D_SOD-123F")
-    (property "LCSC" "C236132")
-    (property "MOUSER" "863-MBR120ESFT1G")
-    (property "MPN" "MBR120ESFT1G")
+    (property "LCSC" "C894433")
+    (property "MOUSER" "512-SS24FL")
+    (property "MPN" "SS24FL")
     (property "Sheetfile" "SW3F1 - Front Panel.kicad_sch")
     (property "Sheetname" "")
@@
       (effects (font (size 1 1) (thickness 0.15)) (justify mirror))
     )
-    (fp_text value "MBR120" (at 0 -2.1) (layer "B.Fab")
+    (fp_text value "SS24FL" (at 0 -2.1) (layer "B.Fab")
       (effects (font (size 1 1) (thickness 0.15)) (justify mirror))
     )
