File: kicad/SW3X1 - Driver Board/SW3X1 - Driver Board.kicad_sch (KiCad schematic)
At the start: 39 parts, among them J1 SERIAL (3v3), J2 PWR, J3 CONTROL, J4 Channel 1, J5 Channel 2, J6 Channel 3, J7 Channel 4, J8 CH_OUT, U1 TPS5430DDA, U2 Pico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

Commit message: finalize driver board
Parts:
- NT1, TP1, TP2, TP4: now left out of the parts list
Changed lines of the file:
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@@
   )
   (symbol (lib_id "Connector:TestPoint_Small") (at 173.99 113.03 0) (unit 1)
-    (in_bom yes) (on_board yes) (fields_autoplaced)
+    (in_bom no) (on_board yes) (fields_autoplaced)
     (property "Reference" "TP4" (id 0) (at 175.26 111.7599 0)
       (effects (font (size 1.27 1.27)) (justify left))
@@
   )
   (symbol (lib_id "Connector:TestPoint_Small") (at 77.47 33.02 0) (unit 1)
-    (in_bom yes) (on_board yes) (fields_autoplaced)
+    (in_bom no) (on_board yes) (fields_autoplaced)
     (property "Reference" "TP1" (id 0) (at 78.74 31.7499 0)
       (effects (font (size 1.27 1.27)) (justify left))
@@
   )
   (symbol (lib_id "Device:NetTie_2") (at 22.86 40.64 0) (mirror y) (unit 1)
-    (in_bom yes) (on_board yes)
+    (in_bom no) (on_board yes)
     (property "Reference" "NT1" (id 0) (at 22.86 36.83 0))
     (property "Value" "2 mm" (id 1) (at 22.86 39.37 0))
@@
   )
   (symbol (lib_id "Connector:TestPoint_Small") (at 114.3 181.61 0) (unit 1)
-    (in_bom yes) (on_board yes)
+    (in_bom no) (on_board yes)
     (property "Reference" "TP2" (id 0) (at 113.03 180.34 0)
       (effects (font (size 1.27 1.27)) (justify right))

Commit message: fix wrong ADC footprint
Parts:
- JP1: now left out of the parts list
- U4: footprint Package_SO:TSSOP-10_3x3mm_P0.5mm -> Package_SO:VSSOP-10_3x3mm_P0.5mm
Changed lines of the file:
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@@
   )
   (symbol (lib_id "Jumper:SolderJumper_2_Open") (at 26.67 118.11 270) (unit 1)
-    (in_bom yes) (on_board yes) (fields_autoplaced)
+    (in_bom no) (on_board yes) (fields_autoplaced)
     (property "Reference" "JP1" (id 0) (at 24.13 116.8399 90)
       (effects (font (size 1.27 1.27)) (justify right))
@@
       (effects (font (size 1.27 1.27)) (justify right))
     )
-    (property "Footprint" "Package_SO:TSSOP-10_3x3mm_P0.5mm" (id 2) (at 189.23 130.81 0)
+    (property "Footprint" "Package_SO:VSSOP-10_3x3mm_P0.5mm" (id 2) (at 189.23 130.81 0)
       (effects (font (size 1.27 1.27)) hide)
     )
@@
     )
     (path "/2e328f1e-bcfb-4390-842b-9c38fa3ad29a"
-      (reference "U4") (unit 1) (value "ADS1015") (footprint "Package_SO:TSSOP-10_3x3mm_P0.5mm")
-    )
-  )
+      (reference "U4") (unit 1) (value "ADS1015") (footprint "Package_SO:VSSOP-10_3x3mm_P0.5mm")
+    )
+  )

Commit message: misc. cleanup
Parts:
- R9: value 1.5K -> 4.7K; LCSC C114668 -> C99782; MOUSER 603-RC0603FR-071K5L -> 603-RC0603FR-074K7L; MPN RC0603FR-071K5L -> RC0603FR-074K7L
Connections:
- net +9V: now also R9.1; no longer R9.2
- net VIN: now also C1.2, C2.2, J2.1 (Pin_1), J2.2 (Pin_2), U1.7 (VIN); no longer D3.2 (A), J3.2 (Pin_2), JP1.1 (A)
- net Vdrive: no longer C1.2, C2.2, J2.1 (Pin_1), J2.2 (Pin_2), U1.7 (VIN)
- net at D4.2 (A): now also R9.2; no longer R9.1
- new net VDD: D3.2 (A), J3.2 (Pin_2), JP1.1 (A)

Commit message: simplify bom - use SS24FL
Parts:
- D3: value DSS14 -> SS24FL; LCSC C511864 -> C894433; MOUSER 241-SS1040FLR100001 -> 512-SS24FL; MPN (none) -> SS24FL
Changed lines of the file:
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@@
   (title_block
     (title "SW3X1 - Driver Board")
-    (date "2022-08-19")
+    (date "2022-12-21")
     (rev "1")
     (company "saawsm")
@@
     (in_bom yes) (on_board yes)
     (property "Reference" "D3" (id 0) (at 144.78 82.55 0))
-    (property "Value" "DSS14" (id 1) (at 144.78 85.09 0))
+    (property "Value" "SS24FL" (id 1) (at 144.78 85.09 0))
     (property "Footprint" "Diode_SMD:D_SOD-123F" (id 2) (at 144.78 88.9 0)
       (effects (font (size 1.27 1.27)) hide)
@@
       (effects (font (size 1.27 1.27)) hide)
     )
-    (property "LCSC" "C511864" (id 4) (at 144.78 88.9 0)
+    (property "LCSC" "C894433" (id 4) (at 144.78 88.9 0)
       (effects (font (size 1.27 1.27)) hide)
     )
-    (property "MOUSER" "241-SS1040FLR100001" (id 5) (at 144.78 88.9 0)
+    (property "MOUSER" "512-SS24FL" (id 5) (at 144.78 88.9 0)
+      (effects (font (size 1.27 1.27)) hide)
+    )
+    (property "MPN" "SS24FL" (id 6) (at 144.78 88.9 0)
       (effects (font (size 1.27 1.27)) hide)
     )
@@
     )
     (path "/6fd387ea-d867-4148-9535-8d3a66d97fd9"
-      (reference "D3") (unit 1) (value "DSS14") (footprint "Diode_SMD:D_SOD-123F")
+      (reference "D3") (unit 1) (value "SS24FL") (footprint "Diode_SMD:D_SOD-123F")
     )
     (path "/92dfd66b-264f-4156-9a98-4fda7049ad7f"

Commit message: fix incorrect MPN
Parts:
- D1: MOUSER 710-150060BS75000 -> 710-150060VS75000; MPN 150060BS75000 -> 150060VS75000
Other:
- moved on the sheet: J1, J2, JP1, R1, R2, R3
