File: kicad/output/SW3O1/SW3O1.kicad_pcb (KiCad board)
At the start: 2 copper layers, 65 x 24.6 mm, 36 parts, among them Q1 NTF2955T1G, Q2 DMN2041L, Q3 DMN2041L, T1 42TL004-RC, U1 SW-32MO, U2 LM358ADT

Commit message: cleanup
Parts:
- removed C10: DNP, Capacitor_SMD:C_0603_1608Metric
- removed the R9 at (129.3, 75.9)
- R3: value 3K -> 2K
- renumbered R11 to R10, R12 to R11, R13 to R12, R14 to R13, R10 to R9
Routing:
- net Net-(C9-Pad2): track 17.8 -> 17.0 mm

Commit message: simplify bom - use SS24FL
Parts:
- D2, D3: value DSS14UTR -> SS24FL
Changed lines of the file:
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@@
     (descr "D_SOD-123F")
     (tags "D_SOD-123F")
-    (property "MPN" "DSS14U")
+    (property "LCSC" "C894433")
+    (property "MOUSER" "512-SS24FL")
+    (property "MPN" "SS24FL")
     (property "Sheetfile" "SW3O1.kicad_sch")
     (property "Sheetname" "")
@@
       (effects (font (size 1 1) (thickness 0.15)))
     )
-    (fp_text value "DSS14UTR" (at -3.526104 0.921393 180) (layer "F.Fab")
+    (fp_text value "SS24FL" (at -3.526104 0.921393 180) (layer "F.Fab")
       (effects (font (size 1 1) (thickness 0.15)))
     )
@@
     (descr "D_SOD-123F")
     (tags "D_SOD-123F")
-    (property "MPN" "DSS14U")
+    (property "LCSC" "C894433")
+    (property "MOUSER" "512-SS24FL")
+    (property "MPN" "SS24FL")
     (property "Sheetfile" "SW3O1.kicad_sch")
     (property "Sheetname" "")
@@
       (effects (font (size 1 1) (thickness 0.15)))
     )
-    (fp_text value "DSS14UTR" (at -3.61446 -1.987404 180) (layer "F.Fab")
+    (fp_text value "SS24FL" (at -3.61446 -1.987404 180) (layer "F.Fab")
       (effects (font (size 1 1) (thickness 0.15)))
     )
