File: kicad/output/SW3O2/SW3O2.kicad_pcb (KiCad board)
At the start: 2 copper layers, 65 x 24.6 mm, 33 parts, among them Q1 IRF9Z24NPBF, Q2 DMN2041L, Q3 DMN2041L, T1 42TL004-RC, U1 SW-32MO, U2 LM358ADT

Commit message: simplify bom - use SS24FL
Parts:
- D2, D3: value DSS14UTR -> SS24FL
Changed lines of the file:
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@@
     (descr "D_SOD-123F")
     (tags "D_SOD-123F")
-    (property "MPN" "DSS14U")
+    (property "MPN" "SS24FL")
     (property "Sheetfile" "SW3O2.kicad_sch")
     (property "Sheetname" "")
@@
       (effects (font (size 1 1) (thickness 0.15)))
     )
-    (fp_text value "DSS14UTR" (at -3.526104 0.921393) (layer "F.Fab")
+    (fp_text value "SS24FL" (at -3.526104 0.921393) (layer "F.Fab")
       (effects (font (size 1 1) (thickness 0.15)))
     )
@@
     (descr "D_SOD-123F")
     (tags "D_SOD-123F")
-    (property "MPN" "DSS14U")
+    (property "MPN" "SS24FL")
     (property "Sheetfile" "SW3O2.kicad_sch")
     (property "Sheetname" "")
@@
       (effects (font (size 1 1) (thickness 0.15)))
     )
-    (fp_text value "DSS14UTR" (at -3.61446 -1.987404) (layer "F.Fab")
+    (fp_text value "SS24FL" (at -3.61446 -1.987404) (layer "F.Fab")
       (effects (font (size 1 1) (thickness 0.15)))
     )
