File: kicad/output/SW3O2/SW3O2.kicad_sch (KiCad schematic)
At the start: 33 parts, among them Q1 IRF9Z24NPBF, Q2 DMN2041L, Q3 DMN2041L, T1 42TL004-RC, U1 SW-32MO, U2 LM358ADT

Commit message: simplify bom - use SS24FL
Parts:
- D2, D3: value DSS14UTR -> SS24FL; MPN DSS14U -> SS24FL
Changed lines of the file:
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@@
   (title_block
     (title "SW3O2")
-    (date "2022-11-09")
+    (date "2022-12-23")
     (rev "1")
     (company "saawsm")
@@
   (symbol (lib_id "Transistor_FET:DMN2041L") (at 218.44 81.28 0) (unit 1)
     (in_bom yes) (on_board yes)
-    (property "Reference" "Q2" (id 0) (at 224.79 73.66 0)
-      (effects (font (size 1.27 1.27)) (justify left))
-    )
-    (property "Value" "DMN2041L" (id 1) (at 224.79 76.2 0)
+    (property "Reference" "Q2" (id 0) (at 224.79 80.01 0)
+      (effects (font (size 1.27 1.27)) (justify left))
+    )
+    (property "Value" "DMN2041L" (id 1) (at 224.79 82.55 0)
       (effects (font (size 1.27 1.27)) (justify left))
     )
@@
     (in_bom yes) (on_board yes) (fields_autoplaced)
     (property "Reference" "D3" (id 0) (at 200.3425 40.64 0))
-    (property "Value" "DSS14UTR" (id 1) (at 200.3425 43.18 0))
+    (property "Value" "SS24FL" (id 1) (at 200.3425 43.18 0))
     (property "Footprint" "Diode_SMD:D_SOD-123F" (id 2) (at 200.66 36.83 0)
       (effects (font (size 1.27 1.27)) hide)
@@
       (effects (font (size 1.27 1.27)) hide)
     )
-    (property "MPN" "DSS14U" (id 4) (at 200.66 36.83 0)
+    (property "MPN" "SS24FL" (id 4) (at 200.66 36.83 0)
       (effects (font (size 1.27 1.27)) hide)
     )
@@
     (in_bom yes) (on_board yes) (fields_autoplaced)
     (property "Reference" "D2" (id 0) (at 200.3425 20.32 0))
-    (property "Value" "DSS14UTR" (id 1) (at 200.3425 22.86 0))
+    (property "Value" "SS24FL" (id 1) (at 200.3425 22.86 0))
     (property "Footprint" "Diode_SMD:D_SOD-123F" (id 2) (at 200.66 26.67 0)
       (effects (font (size 1.27 1.27)) hide)
@@
       (effects (font (size 1.27 1.27)) hide)
     )
-    (property "MPN" "DSS14U" (id 4) (at 200.66 26.67 0)
+    (property "MPN" "SS24FL" (id 4) (at 200.66 26.67 0)
       (effects (font (size 1.27 1.27)) hide)
     )
@@
     )
     (path "/fb44cdac-4dd3-4941-896e-479910f28a69"
-      (reference "D2") (unit 1) (value "DSS14UTR") (footprint "Diode_SMD:D_SOD-123F")
+      (reference "D2") (unit 1) (value "SS24FL") (footprint "Diode_SMD:D_SOD-123F")
     )
     (path "/4abcd740-c754-47a0-9473-c44600c69288"
-      (reference "D3") (unit 1) (value "DSS14UTR") (footprint "Diode_SMD:D_SOD-123F")
+      (reference "D3") (unit 1) (value "SS24FL") (footprint "Diode_SMD:D_SOD-123F")
     )
     (path "/09c41a12-7105-4f5b-ba67-01f5510a9d75"
